File: 8086 schematics and pcb/8086 schematics and pcb.kicad_pcb (KiCad board)
At the start: 2 copper layers, 3 parts, among them U1 P8086-2, U2 ATmega328P-A

Commit message: initial PCB layout with almost accurate footprints
Parts:
- added D1: LED_Filled, LED_SMD:LED_0603_1608Metric_Pad1.05x0.95mm_HandSolder, F.Cu at (83.7, 63.5)
- added D10: LED_Filled, LED_SMD:LED_0603_1608Metric_Pad1.05x0.95mm_HandSolder, F.Cu at (83.7, 57.9)
- added D11: LED_Filled, LED_SMD:LED_0603_1608Metric_Pad1.05x0.95mm_HandSolder, F.Cu at (83.7, 46.7)
- added D12: LED_Filled, LED_SMD:LED_0603_1608Metric_Pad1.05x0.95mm_HandSolder, F.Cu at (83.7, 41.1)
- added D13: LED_Filled, LED_SMD:LED_0603_1608Metric_Pad1.05x0.95mm_HandSolder, F.Cu at (83.7, 29.8)
- added D14: LED_Filled, LED_SMD:LED_0603_1608Metric_Pad1.05x0.95mm_HandSolder, F.Cu at (174.6, 58.3)
- added D15: LED_Filled, LED_SMD:LED_0603_1608Metric_Pad1.05x0.95mm_HandSolder, F.Cu at (174.6, 55.4)
- added D16: LED_Filled, LED_SMD:LED_0603_1608Metric_Pad1.05x0.95mm_HandSolder, F.Cu at (174.6, 43.5)
- added D17: LED_Filled, LED_SMD:LED_0603_1608Metric_Pad1.05x0.95mm_HandSolder, F.Cu at (174.6, 37.6)
- added D18: LED_Filled, LED_SMD:LED_0603_1608Metric_Pad1.05x0.95mm_HandSolder, F.Cu at (174.6, 28.7)
- added D19: LED_Filled, LED_SMD:LED_0603_1608Metric_Pad1.05x0.95mm_HandSolder, F.Cu at (83.9, 66.3)
- added D2: LED_Filled, LED_SMD:LED_0603_1608Metric_Pad1.05x0.95mm_HandSolder, F.Cu at (83.7, 52.3)
- added D20: LED_Filled, LED_SMD:LED_0603_1608Metric_Pad1.05x0.95mm_HandSolder, F.Cu at (83.7, 49.5)
- added D21: LED_Filled, LED_SMD:LED_0603_1608Metric_Pad1.05x0.95mm_HandSolder, F.Cu at (83.7, 43.9)
- added D22: LED_Filled, LED_SMD:LED_0603_1608Metric_Pad1.05x0.95mm_HandSolder, F.Cu at (83.7, 27.0)
- added D23: LED_Filled, LED_SMD:LED_0603_1608Metric_Pad1.05x0.95mm_HandSolder, F.Cu at (174.6, 61.3)
- added D24: LED_Filled, LED_SMD:LED_0603_1608Metric_Pad1.05x0.95mm_HandSolder, F.Cu at (174.6, 49.4)
- added D25: LED_Filled, LED_SMD:LED_0603_1608Metric_Pad1.05x0.95mm_HandSolder, F.Cu at (174.6, 40.6)
- added D26: LED_Filled, LED_SMD:LED_0603_1608Metric_Pad1.05x0.95mm_HandSolder, F.Cu at (174.6, 31.7)
- added D27: LED_Filled, LED_SMD:LED_0603_1608Metric_Pad1.05x0.95mm_HandSolder, F.Cu at (174.6, 25.7)
- added D28: LED_Filled, LED_SMD:LED_0603_1608Metric_Pad1.05x0.95mm_HandSolder, F.Cu at (83.7, 60.7)
- added D29: LED_Filled, LED_SMD:LED_0603_1608Metric_Pad1.05x0.95mm_HandSolder, F.Cu at (83.7, 55.1)
- added D3: LED_Filled, LED_SMD:LED_0603_1608Metric_Pad1.05x0.95mm_HandSolder, F.Cu at (83.7, 35.5)
- added D30: LED_Filled, LED_SMD:LED_0603_1608Metric_Pad1.05x0.95mm_HandSolder, F.Cu at (83.7, 38.3)
- added D31: LED_Filled, LED_SMD:LED_0603_1608Metric_Pad1.05x0.95mm_HandSolder, F.Cu at (83.7, 24.2)
- added D32: LED_Filled, LED_SMD:LED_0603_1608Metric_Pad1.05x0.95mm_HandSolder, F.Cu at (174.6, 67.2)
- added D4: LED_Filled, LED_SMD:LED_0603_1608Metric_Pad1.05x0.95mm_HandSolder, F.Cu at (83.7, 32.6)
- added D5: LED_Filled, LED_SMD:LED_0603_1608Metric_Pad1.05x0.95mm_HandSolder, F.Cu at (174.6, 64.3)
- added D6: LED_Filled, LED_SMD:LED_0603_1608Metric_Pad1.05x0.95mm_HandSolder, F.Cu at (174.6, 52.4)
- added D7: LED_Filled, LED_SMD:LED_0603_1608Metric_Pad1.05x0.95mm_HandSolder, F.Cu at (174.6, 46.5)
- added D8: LED_Filled, LED_SMD:LED_0603_1608Metric_Pad1.05x0.95mm_HandSolder, F.Cu at (174.6, 34.6)
- added D9: LED_Filled, LED_SMD:LED_0603_1608Metric_Pad1.05x0.95mm_HandSolder, F.Cu at (174.6, 22.8)
- added R1: 10K, Resistor_SMD:R_0603_1608Metric_Pad0.98x0.95mm_HandSolder, F.Cu at (278.2, 21.6)
- added R10: R_US, Resistor_SMD:R_0603_1608Metric_Pad0.98x0.95mm_HandSolder, F.Cu at (169.9, 50.0)
- added R11: R_US, Resistor_SMD:R_0603_1608Metric_Pad0.98x0.95mm_HandSolder, F.Cu at (169.9, 44.6)
- added R12: R_US, Resistor_SMD:R_0603_1608Metric_Pad0.98x0.95mm_HandSolder, F.Cu at (169.9, 33.7)
- added R13: R_US, Resistor_SMD:R_0603_1608Metric_Pad0.98x0.95mm_HandSolder, F.Cu at (169.9, 30.9)
- added R14: R_US, Resistor_SMD:R_0603_1608Metric_Pad0.98x0.95mm_HandSolder, F.Cu at (88.6, 63.4)
- added R15: R_US, Resistor_SMD:R_0603_1608Metric_Pad0.98x0.95mm_HandSolder, F.Cu at (88.6, 52.2)
- added R16: R_US, Resistor_SMD:R_0603_1608Metric_Pad0.98x0.95mm_HandSolder, F.Cu at (88.6, 41.0)
- added R17: R_US, Resistor_SMD:R_0603_1608Metric_Pad0.98x0.95mm_HandSolder, F.Cu at (88.6, 35.4)
- added R18: R_US, Resistor_SMD:R_0603_1608Metric_Pad0.98x0.95mm_HandSolder, F.Cu at (88.6, 24.1)
- added R19: R_US, Resistor_SMD:R_0603_1608Metric_Pad0.98x0.95mm_HandSolder, F.Cu at (169.9, 52.8)
- added R2: 10K, Resistor_SMD:R_0603_1608Metric_Pad0.98x0.95mm_HandSolder, F.Cu at (278.2, 24.1)
- added R20: R_US, Resistor_SMD:R_0603_1608Metric_Pad0.98x0.95mm_HandSolder, F.Cu at (169.9, 22.5)
- added R21: R_US, Resistor_SMD:R_0603_1608Metric_Pad0.98x0.95mm_HandSolder, F.Cu at (169.9, 39.1)
- added R22: R_US, Resistor_SMD:R_0603_1608Metric_Pad0.98x0.95mm_HandSolder, F.Cu at (169.9, 28.2)
- added R23: R_US, Resistor_SMD:R_0603_1608Metric_Pad0.98x0.95mm_HandSolder, F.Cu at (170.1, 67.2)
- added R24: R_US, Resistor_SMD:R_0603_1608Metric_Pad0.98x0.95mm_HandSolder, F.Cu at (88.6, 57.8)
- added R25: R_US, Resistor_SMD:R_0603_1608Metric_Pad0.98x0.95mm_HandSolder, F.Cu at (88.6, 43.8)
- added R26: R_US, Resistor_SMD:R_0603_1608Metric_Pad0.98x0.95mm_HandSolder, F.Cu at (88.6, 32.6)
- added R27: R_US, Resistor_SMD:R_0603_1608Metric_Pad0.98x0.95mm_HandSolder, F.Cu at (169.9, 60.9)
- added R28: R_US, Resistor_SMD:R_0603_1608Metric_Pad0.98x0.95mm_HandSolder, F.Cu at (169.9, 47.3)
- added R29: R_US, Resistor_SMD:R_0603_1608Metric_Pad0.98x0.95mm_HandSolder, F.Cu at (169.9, 41.9)
- added R3: 10K, Resistor_SMD:R_0603_1608Metric_Pad0.98x0.95mm_HandSolder, F.Cu at (278.2, 26.6)
- added R30: R_US, Resistor_SMD:R_0603_1608Metric_Pad0.98x0.95mm_HandSolder, F.Cu at (169.9, 36.4)
- added R31: R_US, Resistor_SMD:R_0603_1608Metric_Pad0.98x0.95mm_HandSolder, F.Cu at (169.9, 25.5)
- added R32: R_US, Resistor_SMD:R_0603_1608Metric_Pad0.98x0.95mm_HandSolder, F.Cu at (88.6, 60.6)
- added R33: R_US, Resistor_SMD:R_0603_1608Metric_Pad0.98x0.95mm_HandSolder, F.Cu at (88.6, 49.4)
- added R34: R_US, Resistor_SMD:R_0603_1608Metric_Pad0.98x0.95mm_HandSolder, F.Cu at (88.6, 38.2)
- added R35: R_US, Resistor_SMD:R_0603_1608Metric_Pad0.98x0.95mm_HandSolder, F.Cu at (88.6, 27.0)
- added R36: R_US, Resistor_SMD:R_0603_1608Metric_Pad0.98x0.95mm_HandSolder, F.Cu at (169.9, 63.7)
- added R37: R_US, Resistor_SMD:R_0603_1608Metric_Pad0.98x0.95mm_HandSolder, F.Cu at (169.9, 55.5)
- added R4: 10K, Resistor_SMD:R_0603_1608Metric_Pad0.98x0.95mm_HandSolder, F.Cu at (278.2, 29.1)
- added R5: R_US, Resistor_SMD:R_0603_1608Metric_Pad0.98x0.95mm_HandSolder, F.Cu at (88.3, 66.2)
- added R6: R_US, Resistor_SMD:R_0603_1608Metric_Pad0.98x0.95mm_HandSolder, F.Cu at (88.6, 55.0)
- added R7: R_US, Resistor_SMD:R_0603_1608Metric_Pad0.98x0.95mm_HandSolder, F.Cu at (88.6, 46.6)
- added R8: R_US, Resistor_SMD:R_0603_1608Metric_Pad0.98x0.95mm_HandSolder, F.Cu at (88.6, 29.8)
- added R9: R_US, Resistor_SMD:R_0603_1608Metric_Pad0.98x0.95mm_HandSolder, F.Cu at (169.9, 58.2)
- added SW1: SW_Push, Button_Switch_SMD:SW_Push_1P1T_NO_6x6mm_H9.5mm, F.Cu at (147.2, 87.2)
- added SW10: SW_Push, Button_Switch_SMD:SW_Push_1P1T_NO_6x6mm_H9.5mm, F.Cu at (128.7, 98.2)
- added SW11: SW_Push, Button_Switch_SMD:SW_Push_1P1T_NO_6x6mm_H9.5mm, F.Cu at (121.2, 98.2)
- added SW12: SW_Push, Button_Switch_SMD:SW_Push_1P1T_NO_6x6mm_H9.5mm, F.Cu at (113.7, 98.2)
- added SW13: SW_Push, Button_Switch_SMD:SW_Push_1P1T_NO_6x6mm_H9.5mm, F.Cu at (106.2, 98.2)
- added SW14: SW_Push, Button_Switch_SMD:SW_Push_1P1T_NO_6x6mm_H9.5mm, F.Cu at (98.7, 98.2)
- added SW15: SW_Push, Button_Switch_SMD:SW_Push_1P1T_NO_6x6mm_H9.5mm, F.Cu at (162.2, 87.2)
- added SW16: SW_Push, Button_Switch_SMD:SW_Push_1P1T_NO_6x6mm_H9.5mm, F.Cu at (154.7, 87.2)
- added SW17: SW_Push, Button_Switch_SMD:SW_Push_1P1T_NO_6x6mm_H9.5mm, F.Cu at (132.7, 109.2)
- added SW18: SW_Push, Button_Switch_SMD:SW_Push_1P1T_NO_6x6mm_H9.5mm, F.Cu at (125.2, 109.2)
- added SW19: SW_Push, Button_Switch_SMD:SW_Push_1P1T_NO_6x6mm_H9.5mm, F.Cu at (117.7, 109.2)
- added SW2: SW_Push, Button_Switch_SMD:SW_Push_1P1T_NO_6x6mm_H9.5mm, F.Cu at (139.7, 87.2)
- added SW20: SW_Push, Button_Switch_SMD:SW_Push_1P1T_NO_6x6mm_H9.5mm, F.Cu at (110.2, 109.2)
- added SW21: SW_Push, Button_Switch_SMD:SW_Push_1P1T_NO_6x6mm_H9.5mm, F.Cu at (102.7, 109.2)
- added SW22: SW_Push, Button_Switch_SMD:SW_Push_1P1T_NO_6x6mm_H9.5mm, F.Cu at (158.7, 98.2)
- added SW23: SW_Push, Button_Switch_SMD:SW_Push_1P1T_NO_6x6mm_H9.5mm, F.Cu at (151.2, 98.2)
- added SW24: SW_Push, Button_Switch_SMD:SW_Push_1P1T_NO_6x6mm_H9.5mm, F.Cu at (143.7, 98.2)
- added SW25: SW_Push, Button_Switch_SMD:SW_Push_1P1T_NO_6x6mm_H9.5mm, F.Cu at (171.2, 87.2)
- added SW26: SW_Push, Button_Switch_SMD:SW_Push_1P1T_NO_6x6mm_H9.5mm, F.Cu at (94.7, 109.2)
- added SW27: SW_Push, Button_Switch_SMD:SW_Push_1P1T_NO_6x6mm_H9.5mm, F.Cu at (169.4, 98.2)
- added SW28: SW_Push, Button_Switch_SMD:SW_Push_1P1T_NO_6x6mm_H9.5mm, F.Cu at (163.9, 109.2)
- added SW29: SW_Push, Button_Switch_SMD:SW_Push_1P1T_NO_6x6mm_H9.5mm, F.Cu at (89.0, 98.2)
- added SW3: SW_Push, Button_Switch_SMD:SW_Push_1P1T_NO_6x6mm_H9.5mm, F.Cu at (132.2, 87.2)
- added SW30: SW_Push, Button_Switch_SMD:SW_Push_1P1T_NO_6x6mm_H9.5mm, F.Cu at (86.7, 109.2)
- added SW31: SW_Push, Button_Switch_SMD:SW_Push_1P1T_NO_6x6mm_H9.5mm, F.Cu at (147.7, 109.2)
- added SW32: SW_Push, Button_Switch_SMD:SW_Push_1P1T_NO_6x6mm_H9.5mm, F.Cu at (140.2, 109.2)
- added SW4: SW_Push, Button_Switch_SMD:SW_Push_1P1T_NO_6x6mm_H9.5mm, F.Cu at (124.7, 87.2)
- added SW5: SW_Push, Button_Switch_SMD:SW_Push_1P1T_NO_6x6mm_H9.5mm, F.Cu at (117.2, 87.2)
- added SW6: SW_Push, Button_Switch_SMD:SW_Push_1P1T_NO_6x6mm_H9.5mm, F.Cu at (109.7, 87.2)
- added SW7: SW_Push, Button_Switch_SMD:SW_Push_1P1T_NO_6x6mm_H9.5mm, F.Cu at (102.2, 87.2)
- added SW8: SW_Push, Button_Switch_SMD:SW_Push_1P1T_NO_6x6mm_H9.5mm, F.Cu at (94.7, 87.2)
- added SW9: SW_Push, Button_Switch_SMD:SW_Push_1P1T_NO_6x6mm_H9.5mm, F.Cu at (136.2, 98.2)
- added U10: 74HC595, Package_SO:SOIC-16W_7.5x10.3mm_P1.27mm, F.Cu at (222.1, 89.2)
- added U11: 74HC595, Package_SO:SOIC-16W_7.5x10.3mm_P1.27mm, F.Cu at (208.4, 88.8)
- added U12: 74HC595, Package_SO:SOIC-16W_7.5x10.3mm_P1.27mm, F.Cu at (198.6, 75.2)
- added U13: 74HC165, Package_SO:SOIC-16W_7.5x10.3mm_P1.27mm, F.Cu at (210.8, 75.0)
- added U14: 74HC165, Package_SO:SOIC-16W_7.5x10.3mm_P1.27mm, F.Cu at (222.6, 74.8)
- added U15: AMS1117-3.3, Package_TO_SOT_SMD:SOT-223-3_TabPin2, F.Cu at (241.9, 73.7)
- added U16: 74AC373, Package_SO:SOIC-20W_7.5x12.8mm_P1.27mm, F.Cu at (102.2, 44.9)
- added U17: CXK58257AM, Package_SO:SOIC-28W_7.5x17.9mm_P1.27mm, F.Cu at (265.6, 59.8)
- added U18: IS61C256AH, Package_SO:TSOP-I-28_11.8x8mm_P0.55mm, F.Cu at (259.6, 46.2)
- added U19: IS61C256AH, Package_SO:TSOP-I-28_11.8x8mm_P0.55mm, F.Cu at (259.9, 78.4)
- added U20: IS61C3216, Package_SO:TSOP-II-44_10.16x18.41mm_P0.8mm, F.Cu at (266.2, 83.3)
- added U21: IS61C256AH, Package_SO:TSOP-I-28_11.8x8mm_P0.55mm, F.Cu at (259.9, 88.2)
- added U22: AM29F002, Package_SO:TSOP-I-32_18.4x8mm_P0.5mm, F.Cu at (261.6, 33.9)
- added U23: 74HC14, Package_SO:SOIC-14_3.9x8.7mm_P1.27mm, F.Cu at (210.6, 21.3)
- added U24: 28F400, Package_SO:TSOP-I-48_18.4x12mm_P0.5mm, F.Cu at (258.4, 29.5)
- added U25: CP2102N-Axx-xQFN28, Package_DFN_QFN:QFN-28-1EP_5x5mm_P0.5mm_EP3.35x3.35mm, F.Cu at (207.2, 106.5)
- added U26: AM29F002, Package_SO:TSOP-I-32_18.4x8mm_P0.5mm, F.Cu at (262.1, 24.6)
- added U27: 74HC02, Package_SO:SOIC-14_3.9x8.7mm_P1.27mm, F.Cu at (201.3, 21.5)
- added U28: 74AC373, Package_SO:SOIC-20W_7.5x12.8mm_P1.27mm, F.Cu at (101.3, 27.4)
- added U3: 74HC373, Package_SO:SOIC-20W_7.5x12.8mm_P1.27mm, F.Cu at (227.7, 56.1)
- added U30: 74AC00, Package_SO:SOIC-14_3.9x8.7mm_P1.27mm, F.Cu at (160.1, 44.3)
- added U31: 74HC02, Package_SO:SOIC-14_3.9x8.7mm_P1.27mm, F.Cu at (160.4, 27.3)
- added U32: 74AC373, Package_SO:SOIC-20W_7.5x12.8mm_P1.27mm, F.Cu at (116.5, 45.1)
- added U33: 74AC373, Package_SO:SOIC-20W_7.5x12.8mm_P1.27mm, F.Cu at (131.8, 45.5)
- added U34: 74AC373, Package_SO:SOIC-20W_7.5x12.8mm_P1.27mm, F.Cu at (146.0, 45.5)
- added U35: 74AC373, Package_SO:SOIC-20W_7.5x12.8mm_P1.27mm, F.Cu at (117.6, 27.3)
- added U36: 74AC373, Package_SO:SOIC-20W_7.5x12.8mm_P1.27mm, F.Cu at (132.1, 27.2)
- added U37: 74AC373, Package_SO:SOIC-20W_7.5x12.8mm_P1.27mm, F.Cu at (146.0, 28.0)
- added U4: 74HC373, Package_SO:SOIC-20W_7.5x12.8mm_P1.27mm, F.Cu at (212.5, 56.4)
- added U5: 74HC373, Package_SO:SOIC-20W_7.5x12.8mm_P1.27mm, F.Cu at (197.8, 56.0)
- added U6: 74LS138, Package_SO:SOIC-16_3.9x9.9mm_P1.27mm, F.Cu at (233.4, 22.6)
- added U7: 74LS138, Package_SO:SOIC-16_3.9x9.9mm_P1.27mm, F.Cu at (223.1, 22.1)
- added U8: 74AC00, Package_SO:SOIC-14_3.9x8.7mm_P1.27mm, F.Cu at (191.7, 21.6)
- added U9: IS61C256AH, Package_SO:TSOP-I-28_11.8x8mm_P0.55mm, F.Cu at (258.9, 57.5)
- moved U2 161.8 mm to (194.8, 105.8), turned to 90 degrees
- moved U1 84.8 mm to (237.3, 30.5), turned to -90 degrees
- moved BUS1 82.9 mm to (40.6, 60.0)
Connections:
- BUS1 pad 10: unconnected-(BUS1-AD9-Pad10) -> AD9
- BUS1 pad 11: unconnected-(BUS1-AD10-Pad11) -> AD10
- BUS1 pad 12: unconnected-(BUS1-AD11-Pad12) -> AD11
- BUS1 pad 13: unconnected-(BUS1-AD12-Pad13) -> AD12
- BUS1 pad 14: unconnected-(BUS1-AD13-Pad14) -> AD13
- BUS1 pad 15: unconnected-(BUS1-AD14-Pad15) -> AD14
- BUS1 pad 16: unconnected-(BUS1-AD15-Pad16) -> AD15
- BUS1 pad 17: unconnected-(BUS1-A16-Pad17) -> A16
- BUS1 pad 18: unconnected-(BUS1-A17-Pad18) -> A17
- BUS1 pad 19: unconnected-(BUS1-A18-Pad19) -> A18
- BUS1 pad 20: unconnected-(BUS1-A19-Pad20) -> A19
- BUS1 pad 21: unconnected-(BUS1-~{BHE}-Pad21) -> ~{BHE}
- BUS1 pad 22: unconnected-(BUS1-ALE-Pad22) -> BUSALE
- BUS1 pad 23: unconnected-(BUS1-~{RD}-Pad23) -> ~{RD}
- BUS1 pad 24: unconnected-(BUS1-~{WR}-Pad24) -> ~{WR}
- BUS1 pad 25: unconnected-(BUS1-READY-Pad25) -> READY
- BUS1 pad 26: unconnected-(BUS1-~{IO0}-Pad26) -> ~{IO0}
- BUS1 pad 27: unconnected-(BUS1-~{IO1}-Pad27) -> ~{IO1}
- BUS1 pad 28: unconnected-(BUS1-~{IO2}-Pad28) -> ~{IO2}
- BUS1 pad 29: unconnected-(BUS1-~{IO3}-Pad29) -> ~{IO3}
- BUS1 pad 3: AD2 -> AD1
- BUS1 pad 30: unconnected-(BUS1-~{SEG5}-Pad30) -> ~{SEG5}
- BUS1 pad 31: unconnected-(BUS1-~{SEG6}-Pad31) -> ~{SEG6}
- BUS1 pad 32: unconnected-(BUS1-~{SEG7}-Pad32) -> ~{SEG7}
- BUS1 pad 33: unconnected-(BUS1-~{TEST}-Pad33) -> ~{TEST}
- BUS1 pad 34: unconnected-(BUS1-NMI-Pad34) -> NMI
- BUS1 pad 35: unconnected-(BUS1-INTR-Pad35) -> INTR
- BUS1 pad 36: unconnected-(BUS1-~{INTA}-Pad36) -> ~{INTA}
- BUS1 pad 37: unconnected-(BUS1-HOLD-Pad37) -> HOLD
- BUS1 pad 38: unconnected-(BUS1-HLDA-Pad38) -> HLDA
- BUS1 pad 39: unconnected-(BUS1-RESET-Pad39) -> RESET
- BUS1 pad 40: unconnected-(BUS1-CLK-Pad40) -> CLK
- BUS1 pad 41: unconnected-(BUS1-GND-Pad41) -> +5V
- BUS1 pad 42: unconnected-(BUS1-GND-Pad42) -> +5V
- BUS1 pad 43: unconnected-(BUS1-5V-Pad43) -> +3.3V
- BUS1 pad 44: unconnected-(BUS1-5V-Pad44) -> +3.3V
- BUS1 pad 47: unconnected-(BUS1-NC-Pad47) -> GND
- BUS1 pad 48: unconnected-(BUS1-NC-Pad48) -> GND
- BUS1 pad 49: unconnected-(BUS1-~{IO4}-Pad49) -> ~{IO4}
- BUS1 pad 50: unconnected-(BUS1-~{IO5}-Pad50) -> ~{IO5}
- BUS1 pad 51: unconnected-(BUS1-~{IO6}-Pad51) -> ~{IO6}
- BUS1 pad 52: unconnected-(BUS1-~{IO7}-Pad52) -> ~{IO7}
- BUS1 pad 53: unconnected-(BUS1-~{SEG2}-Pad53) -> ~{SEG2}
- BUS1 pad 54: unconnected-(BUS1-~{SEG3}-Pad54) -> ~{SEG3}
- BUS1 pad 55: unconnected-(BUS1-~{SEG4}-Pad55) -> ~{SEG4}
- BUS1 pad 6: unconnected-(BUS1-AD5-Pad6) -> AD5
- BUS1 pad 7: unconnected-(BUS1-AD6-Pad7) -> AD6
- BUS1 pad 8: unconnected-(BUS1-AD7-Pad8) -> AD7
- BUS1 pad 9: unconnected-(BUS1-AD8-Pad9) -> AD8
- U1 pad 1: unconnected-(U1-GND-Pad1) -> GND
- U1 pad 10: unconnected-(U1-AD6-Pad10) -> AD6
- U1 pad 17: unconnected-(U1-NMI-Pad17) -> NMI
- U1 pad 18: unconnected-(U1-INTR-Pad18) -> INTR
- U1 pad 19: unconnected-(U1-CLK-Pad19) -> CLK
- U1 pad 2: unconnected-(U1-AD14-Pad2) -> AD14
- U1 pad 20: unconnected-(U1-GND-Pad20) -> GND
- U1 pad 21: unconnected-(U1-RESET-Pad21) -> RESET
- U1 pad 22: unconnected-(U1-READY-Pad22) -> READY
- U1 pad 23: unconnected-(U1-~{TEST}-Pad23) -> ~{TEST}
- U1 pad 24: unconnected-(U1-~{INTA}-Pad24) -> ~{INTA}
- U1 pad 25: unconnected-(U1-ALE-Pad25) -> /8086 Module - 1/CPUALE
- U1 pad 28: unconnected-(U1-M/~{IO}-Pad28) -> /8086 Module - 1/M/~{IO}
- U1 pad 29: unconnected-(U1-~{WR}-Pad29) -> ~{WR}
- U1 pad 3: unconnected-(U1-AD13-Pad3) -> AD13
- U1 pad 30: unconnected-(U1-HLDA-Pad30) -> HLDA
- U1 pad 31: unconnected-(U1-HOLD-Pad31) -> HOLD
- U1 pad 32: unconnected-(U1-~{RD}-Pad32) -> ~{RD}
- U1 pad 33: unconnected-(U1-NM/~{MX}-Pad33) -> +5V
- U1 pad 34: unconnected-(U1-~{BHE}-Pad34) -> ~{BHE}
- U1 pad 35: unconnected-(U1-A19-Pad35) -> A19
- U1 pad 36: unconnected-(U1-A18-Pad36) -> A18
- U1 pad 37: unconnected-(U1-A17-Pad37) -> A17
- U1 pad 38: unconnected-(U1-A16-Pad38) -> A16
- U1 pad 39: unconnected-(U1-AD15-Pad39) -> AD15
- U1 pad 4: unconnected-(U1-AD12-Pad4) -> AD12
- U1 pad 40: unconnected-(U1-V_{CC}-Pad40) -> +5V
- U1 pad 5: unconnected-(U1-AD11-Pad5) -> AD11
- U1 pad 6: unconnected-(U1-AD10-Pad6) -> AD10
- U1 pad 7: unconnected-(U1-AD9-Pad7) -> AD9
- U1 pad 8: unconnected-(U1-AD8-Pad8) -> AD8
- U1 pad 9: unconnected-(U1-AD7-Pad9) -> AD7
- U2 pad 1: unconnected-(U2-PD3-Pad1) -> ~{WR}
- U2 pad 10: unconnected-(U2-PD6-Pad10) -> RESET
- U2 pad 11: unconnected-(U2-PD7-Pad11) -> ~{INTA}
- U2 pad 12: AD0 -> HOLD
- U2 pad 13: AD2 -> HLDA
- U2 pad 14: AD3 -> /Microcontroller Module/REG_RCLK
- U2 pad 15: AD4 -> /Microcontroller Module/SPI_MOSI
- U2 pad 16: AD5 -> /Microcontroller Module/SPI_MISO
- U2 pad 17: unconnected-(U2-PB5-Pad17) -> /Microcontroller Module/SPI_SCK
- U2 pad 18: unconnected-(U2-AVCC-Pad18) -> +5V
- U2 pad 2: unconnected-(U2-PD4-Pad2) -> BUSALE
- U2 pad 21: Net-(U2-GND-Pad21) -> GND
- U2 pad 23: unconnected-(U2-PC0-Pad23) -> /Microcontroller Module/REG_OE
- U2 pad 24: unconnected-(U2-PC1-Pad24) -> /Microcontroller Module/REG_SHLD
- U2 pad 25: unconnected-(U2-PC2-Pad25) -> INTR
- U2 pad 26: unconnected-(U2-PC3-Pad26) -> NMI
- U2 pad 27: unconnected-(U2-PC4-Pad27) -> ~{TEST}
- U2 pad 28: unconnected-(U2-PC5-Pad28) -> READY
- U2 pad 3: Net-(U2-GND-Pad21) -> GND
- U2 pad 32: unconnected-(U2-PD2-Pad32) -> ~{RD}
- U2 pad 4: Net-(U2-VCC-Pad4) -> +5V
- U2 pad 5: Net-(U2-GND-Pad21) -> GND
- U2 pad 6: Net-(U2-VCC-Pad4) -> +5V
- U2 pad 9: unconnected-(U2-PD5-Pad9) -> CLK
Routing:
- net AD3: track 167.4 -> 25.2 mm, vias 4 -> 0
- net AD0: track 126.9 -> 21.1 mm, vias 4 -> 0
- net AD2: track 121.8 -> 24.3 mm, vias 4 -> 0
- net AD4: track 115.7 -> 26.6 mm
- net AD5: track 112.2 -> 27.6 mm
- net /8086 Module - 1/LA2: track 0.00 -> 61.6 mm
- net AD6: track 0.00 -> 61.0 mm
- net /8086 Module - 1/LA3: track 0.00 -> 57.6 mm
- net /8086 Module - 1/LA1: track 0.00 -> 57.4 mm
- net /8086 Module - 1/LA4: track 0.00 -> 48.8 mm
- net ~{RD}: track 0.00 -> 32.8 mm
- net /8086 Module - 1/LA11: track 0.00 -> 32.6 mm
- net AD1: track 54.9 -> 23.2 mm, vias 2 -> 0
- net AD7: track 0.00 -> 31.3 mm
- net /8086 Module - 2/~{MEM1L}: track 0.00 -> 31.2 mm
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Other:
- board outline added: 203.3 x 100 mm
- board text added: "Alt"
- board text added: "Backspcae"
- board text added: "Ctrl"
- board text added: "Enter"
- board text added: "LEDs"
- board text added: "RGB LCD"
- board text added: "Shift"
- board text added: "Space"
