File: 8086 schematics and pcb/module_8086_2.kicad_sch (KiCad schematic)
At the start: 10 parts, among them U17 AM29F002, U18 AM29F002, U19 CXK58257AM, U20 IS61C3216, U21 IS61C256AH, U22 IS61C256AH, U30 IS61C256AH, U31 IS61C256AH, U9 28F400

Commit message: initial PCB layout with almost accurate footprints
Parts:
- U17, U18: footprint (none) -> Package_SO:TSOP-I-32_18.4x8mm_P0.5mm
- U19: footprint (none) -> Package_SO:SOIC-28W_7.5x17.9mm_P1.27mm
- U20: footprint (none) -> Package_SO:TSOP-II-44_10.16x18.41mm_P0.8mm
- U9: footprint Package_SO:PSOP-44_16.9x27.17mm_P1.27mm -> Package_SO:TSOP-I-48_18.4x12mm_P0.5mm
Changed lines of the file:
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@@
       (effects (font (size 1.27 1.27)) (justify left))
     )
-    (property "Footprint" "" (at 35.56 135.89 0)
+    (property "Footprint" "Package_SO:TSOP-I-32_18.4x8mm_P0.5mm" (at 35.56 135.89 0)
       (effects (font (size 1.27 1.27)) hide)
     )
@@
       (effects (font (size 1.27 1.27)) (justify left))
     )
-    (property "Footprint" "" (at 76.2 31.75 0)
+    (property "Footprint" "Package_SO:SOIC-28W_7.5x17.9mm_P1.27mm" (at 76.2 31.75 0)
       (effects (font (size 1.27 1.27)) hide)
     )
@@
       (effects (font (size 1.27 1.27)) (justify left))
     )
-    (property "Footprint" "Package_SO:PSOP-44_16.9x27.17mm_P1.27mm" (at 129.54 133.35 0)
+    (property "Footprint" "Package_SO:TSOP-I-48_18.4x12mm_P0.5mm" (at 129.54 133.35 0)
       (effects (font (size 1.27 1.27)) hide)
     )
@@
       (effects (font (size 1.27 1.27)) (justify left))
     )
-    (property "Footprint" "" (at 76.2 135.89 0)
+    (property "Footprint" "Package_SO:TSOP-I-32_18.4x8mm_P0.5mm" (at 76.2 135.89 0)
       (effects (font (size 1.27 1.27)) hide)
     )
@@
       (effects (font (size 1.27 1.27)) (justify left))
     )
-    (property "Footprint" "" (at 259.08 31.75 0)
-      (effects (font (size 1.27 1.27)) hide)
-    )
+    (property "Footprint" "Package_SO:TSOP-II-44_10.16x18.41mm_P0.8mm" (at 259.08 31.75 0)
+      (effects (font (size 1.27 1.27)) hide)
+    )
