File: 8086 schematics and pcb/module_io.kicad_sch (KiCad schematic)
At the start: 0 parts

Commit message: basic start for IO module
Parts:
- added D1, D10, D11, D12, D13, D14, D15, D16, D17, D18, D19, D2, D20, D21, D22, D23, D24, D25, D26, D27, D28, D29, D3, D30, D31, D32, D4, D5, D6, D7, D8, D9: LED_Filled, symbol Device:LED_Filled
- added JP4: Jumper_2_Bridged, symbol Jumper:Jumper_2_Bridged
- added R10, R11, R12, R13, R14, R15, R16, R17, R18, R19, R20, R21, R22, R23, R24, R25, R26, R27, R28, R29, R30, R31, R32, R33, R34, R35, R36, R37, R5, R6, R7, R8, R9: R_US, symbol Device:R_US
- added SW1, SW10, SW11, SW12, SW13, SW14, SW15, SW16, SW17, SW18, SW19, SW2, SW20, SW21, SW22, SW23, SW24, SW25, SW26, SW27, SW28, SW29, SW3, SW30, SW31, SW32, SW4, SW5, SW6, SW7, SW8, SW9: SW_Push, symbol Switch:SW_Push
- added U16, U28, U32, U33, U34, U35, U36, U37: 74AC373, symbol 8086PC:74AC373
- added U30: 74AC00, symbol 8086PC:74AC00
- added U31: 74HC02, symbol 8086PC:74HC02
Connections:
- new net: JP4.2 (B), U16.11 (LE), U32.11 (LE), U33.11 (LE), U34.11 (LE)
- new net: SW13.2, U32.13 (D4)
- new net: SW14.2, U32.14 (D5)
- new net: SW15.2, U32.17 (D6)
- new net: SW16.2, U32.18 (D7)
- new net: SW9.2, U32.3 (D0)
- new net: SW10.2, U32.4 (D1)
- new net: SW11.2, U32.7 (D2)
- new net: SW12.2, U32.8 (D3)
- new net: SW24.2, U33.18 (D7)
- new net: U30.4, U30.5, U31.4
- new net: SW17.2, U33.3 (D0)
- new net: D5.1 (K), R6.1
- new net: D5.2 (A), U28.12 (O4)
- new net: D19.1 (K), R22.1
- new net: D23.1 (K), R24.1
- new net: D23.2 (A), U36.9 (O3)
- new net: D4.1 (K), R5.1
- new net: D4.2 (A), U28.9 (O3)
- new net: D31.1 (K), R32.1
- new net: D31.2 (A), U37.9 (O3)
- new net: SW25.2, U34.3 (D0)
- new net: D11.1 (K), R14.1
- new net: D24.1 (K), R28.1
- new net: D3.1 (K), R12.1
- new net: D3.2 (A), U28.2 (O0)
- new net: D16.1 (K), R20.1
- new net: SW27.2, U34.7 (D2)
- new net: D27.1 (K), R30.1
- new net: D27.2 (A), U37.5 (O1)
- new net: D10.2 (A), U35.12 (O4)
- new net: D12.2 (A), U35.15 (O5)
- new net: D14.2 (A), U35.16 (O6)
- new net: D16.2 (A), U35.19 (O7)
- new net: D9.2 (A), U35.2 (O0)
- new net: D11.2 (A), U35.5 (O1)
- new net: D13.2 (A), U35.6 (O2)
- new net: D15.2 (A), U35.9 (O3)
- new net: D19.2 (A), U36.5 (O1)
- new net: SW5.2, U16.13 (D4)
- new net: SW2.2, U16.4 (D1)
- new net: D17.1 (K), R21.1
- new net: D9.1 (K), R13.1
- new net: D20.1 (K), R26.1
- new net: D20.2 (A), U36.15 (O5)
- new net: SW31.2, U34.17 (D6)
- new net: D7.1 (K), R8.1
- new net: D7.2 (A), U28.16 (O6)
- new net: D12.1 (K), R18.1
- new net: D10.1 (K), R17.1
- new net: D30.1 (K), R35.1
- new net: D13.1 (K), R15.1
- new net: D22.1 (K), R27.1
- new net: D21.1 (K), R23.1
- new net: D15.1 (K), R16.1
- new net: D30.2 (A), U37.16 (O6)
- new net: SW6.2, U16.14 (D5)
- new net: D32.1 (K), R36.1
- new net: SW20.2, U33.8 (D3)
- new net: SW7.2, U16.17 (D6)
- new net: D26.1 (K), R33.1
- new net: D26.2 (A), U37.12 (O4)
- new net: R37.1, SW8.2, U16.18 (D7)
- new net: SW29.2, U34.13 (D4)
- new net: SW30.2, U34.14 (D5)
- new net: SW32.2, U34.18 (D7)
- new net: SW26.2, U34.4 (D1)
- new net: SW28.2, U34.8 (D3)
- new net: D2.1 (K), R10.1
- new net: SW23.2, U33.17 (D6)
- new net: D8.1 (K), R9.1
- new net: D25.1 (K), R29.1
- new net: D25.2 (A), U37.2 (O0)
- new net: D1.1 (K), R11.1
- new net: D6.2 (A), U28.15 (O5)
- new net: D8.2 (A), U28.19 (O7)
- new net: D1.2 (A), U28.5 (O1)
- new net: D2.2 (A), U28.6 (O2)
- new net: D28.1 (K), R34.1
- new net: D17.2 (A), U36.2 (O0)
- new net: D22.2 (A), U36.16 (O6)
- new net: SW18.2, U33.4 (D1)
- new net: D28.2 (A), U37.15 (O5)
- new net: SW3.2, U16.7 (D2)
- new net: D14.1 (K), R19.1
- new net: D29.1 (K), R31.1
- new net: D32.2 (A), U37.19 (O7)
- new net: D18.1 (K), R25.1
- new net: U30.1, U30.2, U31.1
- new net: SW21.2, U33.13 (D4)
- new net: SW4.2, U16.8 (D3)
- new net: SW22.2, U33.14 (D5)
- new net: SW19.2, U33.7 (D2)
- new net: D6.1 (K), R7.1
- new net: D18.2 (A), U36.12 (O4)
- new net: D21.2 (A), U36.6 (O2)
- new net: D24.2 (A), U36.19 (O7)
- new net: SW1.2, U16.3 (D0)
- new net: D29.2 (A), U37.6 (O2)
- new net +5V: JP4.1 (A), SW1.1, SW10.1, SW11.1, SW12.1, SW13.1, SW14.1, SW15.1, SW16.1, SW17.1, SW18.1, SW19.1, SW2.1, SW20.1, SW21.1, SW22.1, SW23.1, SW24.1, SW25.1, SW26.1, SW27.1, SW28.1, SW29.1, SW3.1, SW30.1, SW31.1, SW32.1, SW4.1, SW5.1, SW6.1, SW7.1, SW8.1, SW9.1, U16.20 (VCC), U28.20 (VCC), U30.14 (V_{CC}), U31.14 (V_{CC}), U32.20 (VCC), U33.20 (VCC), U34.20 (VCC), U35.20 (VCC), U36.20 (VCC), U37.20 (VCC)
- new net AD0: U16.2 (O0), U28.3 (D0), U33.2 (O0), U36.3 (D0)
- new net AD1: U16.5 (O1), U28.4 (D1), U33.5 (O1), U36.4 (D1)
- new net AD10: U32.6 (O2), U34.6 (O2), U35.7 (D2), U37.7 (D2)
- new net AD11: U32.9 (O3), U34.9 (O3), U35.8 (D3), U37.8 (D3)
- new net AD12: U32.12 (O4), U34.12 (O4), U35.13 (D4), U37.13 (D4)
- new net AD13: U32.15 (O5), U34.15 (O5), U35.14 (D5), U37.14 (D5)
- new net AD14: U32.16 (O6), U34.16 (O6), U35.17 (D6), U37.17 (D6)
- new net AD15: U32.19 (O7), U34.19 (O7), U35.18 (D7), U37.18 (D7)
- new net AD2: U16.6 (O2), U28.7 (D2), U33.6 (O2), U36.7 (D2)
- new net AD3: U16.9 (O3), U28.8 (D3), U33.9 (O3), U36.8 (D3)
- new net AD4: U16.12 (O4), U28.13 (D4), U33.12 (O4), U36.13 (D4)
- new net AD5: U16.15 (O5), U28.14 (D5), U33.15 (O5), U36.14 (D5)
- new net AD6: U16.16 (O6), U28.17 (D6), U33.16 (O6), U36.17 (D6)
- new net AD7: U16.19 (O7), U28.18 (D7), U33.19 (O7), U36.18 (D7)
- new net AD8: U32.2 (O0), U34.2 (O0), U35.3 (D0), U37.3 (D0)
- new net AD9: U32.5 (O1), U34.5 (O1), U35.4 (D1), U37.4 (D1)
- new net GND: R10.2, R11.2, R12.2, R13.2, R14.2, R15.2, R16.2, R17.2, R18.2, R19.2, R20.2, R21.2, R22.2, R23.2, R24.2, R25.2, R26.2, R27.2, R28.2, R29.2, R30.2, R31.2, R32.2, R33.2, R34.2, R35.2, R36.2, R37.2, R5.2, R6.2, R7.2, R8.2, R9.2, U16.10 (GND), U28.1 (~{OE}), U28.10 (GND), U30.7 (GND), U31.7 (GND), U32.10 (GND), U33.10 (GND), U34.10 (GND), U35.1 (~{OE}), U35.10 (GND), U36.1 (~{OE}), U36.10 (GND), U37.1 (~{OE}), U37.10 (GND)
- new net WR0: U28.11 (LE), U31.10, U35.11 (LE)
- new net WR1: U31.13, U36.11 (LE), U37.11 (LE)
- new net ~{IO0}: U31.3, U31.9
- new net ~{IO1}: U31.12, U31.6
- new net ~{RD0}: U16.1 (~{OE}), U30.3, U32.1 (~{OE})
- new net ~{RD1}: U30.6, U33.1 (~{OE}), U34.1 (~{OE})
- new net ~{RD}: U31.2, U31.5
- new net ~{WR}: U31.11, U31.8
- no-connect marks 0 -> 6
Other:
- note added: "Character LCD connector"
- note added: "RGB LCD socket"

Commit message: initial PCB layout with almost accurate footprints
Parts:
- D1, D10, D11, D12, D13, D14, D15, D16, D17, D18, D19, D2, D20, D21, D22, D23, D24, D25, D26, D27, D28, D29, D3, D30, D31, D32, D4, D5, D6, D7, D8, D9: footprint (none) -> LED_SMD:LED_0603_1608Metric_Pad1.05x0.95mm_HandSolder
- R10, R11, R12, R13, R14, R15, R16, R17, R18, R19, R20, R21, R22, R23, R24, R25, R26, R27, R28, R29, R30, R31, R32, R33, R34, R35, R36, R37, R5, R6, R7, R8, R9: footprint (none) -> Resistor_SMD:R_0603_1608Metric_Pad0.98x0.95mm_HandSolder
- SW1, SW10, SW11, SW12, SW13, SW14, SW15, SW16, SW17, SW18, SW19, SW2, SW20, SW21, SW22, SW23, SW24, SW25, SW26, SW27, SW28, SW29, SW3, SW30, SW31, SW32, SW4, SW5, SW6, SW7, SW8, SW9: footprint (none) -> Button_Switch_SMD:SW_Push_1P1T_NO_6x6mm_H9.5mm
- U16, U28, U32, U33, U34, U35, U36, U37: footprint (none) -> Package_SO:SOIC-20W_7.5x12.8mm_P1.27mm
- U30, U31: footprint (none) -> Package_SO:SOIC-14_3.9x8.7mm_P1.27mm
