File: 8086 board/8086 board.kicad_pcb (KiCad board)
At the start: 2 copper layers, 100 x 100 mm, 118 parts, among them SW33 SW_Push, U1 74HC02, U10 74HC595, U11 74HC595, U12 74HC595, U13 74HC165, U14 74HC165, U15 AMS1117-3.3, U16 74AC373, U17 CXK58257AM, U18 IS61C256AH, U19 IS61C256AH, U2 ATmega328P-A, U20 IS61C3216, U21 IS61C256AH, U22 AM29F002, U23 74HC14, U24 28F400B5, U25 CP2102N-Axx-xQFN28, U26 AM29F002, U28 74AC373, U3 74AC373, U30 74AC00, U31 74HC02, U32 74AC373, U33 74AC373, U34 74AC373, U35 74AC373, U36 74AC373, U37 74AC373, U4 74AC373, U40 CH340G, U44 P8086-2, U5 74AC373, U6 74HC138, U7 74HC138, U8 74AC00, U9 IS61C256AH

Commit message: initial pcb
Parts:
- removed D33: A4, LED_SMD:LED_0603_1608Metric_Pad1.05x0.95mm_HandSolder
- removed D34: A5, LED_SMD:LED_0603_1608Metric_Pad1.05x0.95mm_HandSolder
- removed D35: A6, LED_SMD:LED_0603_1608Metric_Pad1.05x0.95mm_HandSolder
- removed D36: A7, LED_SMD:LED_0603_1608Metric_Pad1.05x0.95mm_HandSolder
- removed D37: A8, LED_SMD:LED_0603_1608Metric_Pad1.05x0.95mm_HandSolder
- removed D38: A9, LED_SMD:LED_0603_1608Metric_Pad1.05x0.95mm_HandSolder
- removed D39: A10, LED_SMD:LED_0603_1608Metric_Pad1.05x0.95mm_HandSolder
- removed D40: A11, LED_SMD:LED_0603_1608Metric_Pad1.05x0.95mm_HandSolder
- removed D41: A12, LED_SMD:LED_0603_1608Metric_Pad1.05x0.95mm_HandSolder
- removed D42: A13, LED_SMD:LED_0603_1608Metric_Pad1.05x0.95mm_HandSolder
- removed D43: A14, LED_SMD:LED_0603_1608Metric_Pad1.05x0.95mm_HandSolder
- removed D44: A15, LED_SMD:LED_0603_1608Metric_Pad1.05x0.95mm_HandSolder
- removed D45: A16, LED_SMD:LED_0603_1608Metric_Pad1.05x0.95mm_HandSolder
- removed D46: A17, LED_SMD:LED_0603_1608Metric_Pad1.05x0.95mm_HandSolder
- removed D47: A18, LED_SMD:LED_0603_1608Metric_Pad1.05x0.95mm_HandSolder
- removed D48: A0, LED_SMD:LED_0603_1608Metric_Pad1.05x0.95mm_HandSolder
- removed D49: A1, LED_SMD:LED_0603_1608Metric_Pad1.05x0.95mm_HandSolder
- removed D50: A2, LED_SMD:LED_0603_1608Metric_Pad1.05x0.95mm_HandSolder
- removed D51: A3, LED_SMD:LED_0603_1608Metric_Pad1.05x0.95mm_HandSolder
- removed D52: A19, LED_SMD:LED_0603_1608Metric_Pad1.05x0.95mm_HandSolder
- removed D53: ~{BHE}, LED_SMD:LED_0603_1608Metric_Pad1.05x0.95mm_HandSolder
- removed D54: SEG0, LED_SMD:LED_0603_1608Metric_Pad1.05x0.95mm_HandSolder
- removed D55: SEG1, LED_SMD:LED_0603_1608Metric_Pad1.05x0.95mm_HandSolder
- removed D56: PWR, LED_SMD:LED_0603_1608Metric_Pad1.05x0.95mm_HandSolder
- removed U40: CH340G, Package_SO:SOIC-16_3.9x9.9mm_P1.27mm
- removed U44: P8086-2, Package_DIP:DIP-40_W15.24mm
- added C1: 10uF, Capacitor_SMD:C_0603_1608Metric_Pad1.08x0.95mm_HandSolder, F.Cu at (356.4, 20.9)
- added C10: 1uF, Capacitor_SMD:C_0603_1608Metric_Pad1.08x0.95mm_HandSolder, F.Cu at (309.8, 21.3)
- added C11: 1uF, Capacitor_SMD:C_0603_1608Metric_Pad1.08x0.95mm_HandSolder, F.Cu at (309.8, 23.8)
- added C12: 1uF, Capacitor_SMD:C_0603_1608Metric_Pad1.08x0.95mm_HandSolder, F.Cu at (309.8, 26.3)
- added C13: 1uF, Capacitor_SMD:C_0603_1608Metric_Pad1.08x0.95mm_HandSolder, F.Cu at (309.8, 28.8)
- added C14: 1uF, Capacitor_SMD:C_0603_1608Metric_Pad1.08x0.95mm_HandSolder, F.Cu at (309.8, 31.3)
- added C15: 1uF, Capacitor_SMD:C_0603_1608Metric_Pad1.08x0.95mm_HandSolder, F.Cu at (309.8, 33.8)
- added C16: 1uF, Capacitor_SMD:C_0603_1608Metric_Pad1.08x0.95mm_HandSolder, F.Cu at (309.8, 36.3)
- added C17: 1uF, Capacitor_SMD:C_0603_1608Metric_Pad1.08x0.95mm_HandSolder, F.Cu at (314.2, 16.2)
- added C18: 1uF, Capacitor_SMD:C_0603_1608Metric_Pad1.08x0.95mm_HandSolder, F.Cu at (314.2, 18.8)
- added C19: 1uF, Capacitor_SMD:C_0603_1608Metric_Pad1.08x0.95mm_HandSolder, F.Cu at (314.2, 21.3)
- added C2: 10uF, Capacitor_SMD:C_0603_1608Metric_Pad1.08x0.95mm_HandSolder, F.Cu at (356.4, 23.4)
- added C20: 1uF, Capacitor_SMD:C_0603_1608Metric_Pad1.08x0.95mm_HandSolder, F.Cu at (314.2, 23.8)
- added C21: 1uF, Capacitor_SMD:C_0603_1608Metric_Pad1.08x0.95mm_HandSolder, F.Cu at (314.2, 26.3)
- added C22: 1uF, Capacitor_SMD:C_0603_1608Metric_Pad1.08x0.95mm_HandSolder, F.Cu at (314.2, 28.8)
- added C23: 1uF, Capacitor_SMD:C_0603_1608Metric_Pad1.08x0.95mm_HandSolder, F.Cu at (314.2, 31.3)
- added C24: 1uF, Capacitor_SMD:C_0603_1608Metric_Pad1.08x0.95mm_HandSolder, F.Cu at (314.2, 33.8)
- added C25: 1uF, Capacitor_SMD:C_0603_1608Metric_Pad1.08x0.95mm_HandSolder, F.Cu at (314.2, 36.3)
- added C26: 1uF, Capacitor_SMD:C_0603_1608Metric_Pad1.08x0.95mm_HandSolder, F.Cu at (318.5, 16.2)
- added C27: 1uF, Capacitor_SMD:C_0603_1608Metric_Pad1.08x0.95mm_HandSolder, F.Cu at (318.5, 18.8)
- added C28: 1uF, Capacitor_SMD:C_0603_1608Metric_Pad1.08x0.95mm_HandSolder, F.Cu at (318.5, 21.3)
- added C29: 1uF, Capacitor_SMD:C_0603_1608Metric_Pad1.08x0.95mm_HandSolder, F.Cu at (318.5, 23.8)
- added C3: 220uF, Capacitor_Tantalum_SMD:CP_EIA-7343-43_Kemet-X_Pad2.25x2.55mm_HandSolder, F.Cu at (351.1, 16.7)
- added C30: 1uF, Capacitor_SMD:C_0603_1608Metric_Pad1.08x0.95mm_HandSolder, F.Cu at (318.5, 26.3)
- added C31: 1uF, Capacitor_SMD:C_0603_1608Metric_Pad1.08x0.95mm_HandSolder, F.Cu at (318.5, 28.8)
- added C32: 1uF, Capacitor_SMD:C_0603_1608Metric_Pad1.08x0.95mm_HandSolder, F.Cu at (318.5, 31.3)
- added C33: 1uF, Capacitor_SMD:C_0603_1608Metric_Pad1.08x0.95mm_HandSolder, F.Cu at (318.5, 33.8)
- added C34: 1uF, Capacitor_SMD:C_0603_1608Metric_Pad1.08x0.95mm_HandSolder, F.Cu at (318.5, 36.3)
- added C35: 1uF, Capacitor_SMD:C_0603_1608Metric_Pad1.08x0.95mm_HandSolder, F.Cu at (322.9, 16.2)
- added C36: 1uF, Capacitor_SMD:C_0603_1608Metric_Pad1.08x0.95mm_HandSolder, F.Cu at (322.9, 18.8)
- added C37: 1uF, Capacitor_SMD:C_0603_1608Metric_Pad1.08x0.95mm_HandSolder, F.Cu at (322.9, 21.3)
- added C38: 1uF, Capacitor_SMD:C_0603_1608Metric_Pad1.08x0.95mm_HandSolder, F.Cu at (322.9, 23.8)
- added C39: 1uF, Capacitor_SMD:C_0603_1608Metric_Pad1.08x0.95mm_HandSolder, F.Cu at (322.9, 26.3)
- added C4: 1uF, Capacitor_SMD:C_0603_1608Metric_Pad1.08x0.95mm_HandSolder, F.Cu at (334.2, 51.4)
- added C40: 1uF, Capacitor_SMD:C_0603_1608Metric_Pad1.08x0.95mm_HandSolder, F.Cu at (322.9, 28.8)
- added C41: 1uF, Capacitor_SMD:C_0603_1608Metric_Pad1.08x0.95mm_HandSolder, F.Cu at (322.9, 31.3)
- added C42: 1uF, Capacitor_SMD:C_0603_1608Metric_Pad1.08x0.95mm_HandSolder, F.Cu at (322.9, 33.8)
- added C43: 1uF, Capacitor_SMD:C_0603_1608Metric_Pad1.08x0.95mm_HandSolder, F.Cu at (322.9, 36.3)
- added C5: 0.1uF, Capacitor_SMD:C_0603_1608Metric_Pad1.08x0.95mm_HandSolder, F.Cu at (334.2, 53.9)
- added C6: 22pF, Capacitor_SMD:C_0603_1608Metric_Pad1.08x0.95mm_HandSolder, F.Cu at (481.8, 27.3)
- added C7: 22pF, Capacitor_SMD:C_0603_1608Metric_Pad1.08x0.95mm_HandSolder, F.Cu at (481.8, 29.8)
- added C8: 1uF, Capacitor_SMD:C_0603_1608Metric_Pad1.08x0.95mm_HandSolder, F.Cu at (309.8, 16.2)
- added C9: 1uF, Capacitor_SMD:C_0603_1608Metric_Pad1.08x0.95mm_HandSolder, F.Cu at (309.8, 18.8)
- added D1: A0, LED_SMD:LED_0603_1608Metric_Pad1.05x0.95mm_HandSolder, F.Cu at (416.9, 145.3)
- added D10: A9, LED_SMD:LED_0603_1608Metric_Pad1.05x0.95mm_HandSolder, F.Cu at (421.3, 153.1)
- added D11: A10, LED_SMD:LED_0603_1608Metric_Pad1.05x0.95mm_HandSolder, F.Cu at (421.3, 155.6)
- added D12: A11, LED_SMD:LED_0603_1608Metric_Pad1.05x0.95mm_HandSolder, F.Cu at (421.3, 158.2)
- added D13: A12, LED_SMD:LED_0603_1608Metric_Pad1.05x0.95mm_HandSolder, F.Cu at (425.6, 145.3)
- added D14: A13, LED_SMD:LED_0603_1608Metric_Pad1.05x0.95mm_HandSolder, F.Cu at (425.6, 147.9)
- added D15: A14, LED_SMD:LED_0603_1608Metric_Pad1.05x0.95mm_HandSolder, F.Cu at (425.6, 150.5)
- added D16: A15, LED_SMD:LED_0603_1608Metric_Pad1.05x0.95mm_HandSolder, F.Cu at (425.6, 153.1)
- added D17: A16, LED_SMD:LED_0603_1608Metric_Pad1.05x0.95mm_HandSolder, F.Cu at (425.6, 155.6)
- added D18: A17, LED_SMD:LED_0603_1608Metric_Pad1.05x0.95mm_HandSolder, F.Cu at (425.6, 158.2)
- added D19: A18, LED_SMD:LED_0603_1608Metric_Pad1.05x0.95mm_HandSolder, F.Cu at (430.0, 145.3)
- added D2: A1, LED_SMD:LED_0603_1608Metric_Pad1.05x0.95mm_HandSolder, F.Cu at (416.9, 147.9)
- added D20: A19, LED_SMD:LED_0603_1608Metric_Pad1.05x0.95mm_HandSolder, F.Cu at (430.0, 147.9)
- added D21: PWR, LED_SMD:LED_0603_1608Metric_Pad1.05x0.95mm_HandSolder, F.Cu at (430.0, 150.5)
- added D22: ~{BHE}, LED_SMD:LED_0603_1608Metric_Pad1.05x0.95mm_HandSolder, F.Cu at (430.0, 153.1)
- added D23: SEG0, LED_SMD:LED_0603_1608Metric_Pad1.05x0.95mm_HandSolder, F.Cu at (430.0, 155.6)
- added D24: SEG1, LED_SMD:LED_0603_1608Metric_Pad1.05x0.95mm_HandSolder, F.Cu at (430.0, 158.2)
- added D25: LED, LED_SMD:LED_0603_1608Metric_Pad1.05x0.95mm_HandSolder, F.Cu at (399.0, 94.5)
- added D26: LED, LED_SMD:LED_0603_1608Metric_Pad1.05x0.95mm_HandSolder, F.Cu at (399.0, 97.0)
- added D27: LED, LED_SMD:LED_0603_1608Metric_Pad1.05x0.95mm_HandSolder, F.Cu at (399.0, 99.6)
- added D28: LED, LED_SMD:LED_0603_1608Metric_Pad1.05x0.95mm_HandSolder, F.Cu at (399.0, 102.2)
- added D3: A2, LED_SMD:LED_0603_1608Metric_Pad1.05x0.95mm_HandSolder, F.Cu at (416.9, 150.5)
- added D4: A3, LED_SMD:LED_0603_1608Metric_Pad1.05x0.95mm_HandSolder, F.Cu at (416.9, 153.1)
- added D5: A4, LED_SMD:LED_0603_1608Metric_Pad1.05x0.95mm_HandSolder, F.Cu at (416.9, 155.6)
- added D6: A5, LED_SMD:LED_0603_1608Metric_Pad1.05x0.95mm_HandSolder, F.Cu at (416.9, 158.2)
- added D7: A6, LED_SMD:LED_0603_1608Metric_Pad1.05x0.95mm_HandSolder, F.Cu at (421.3, 145.3)
- added D8: A7, LED_SMD:LED_0603_1608Metric_Pad1.05x0.95mm_HandSolder, F.Cu at (421.3, 147.9)
- added D9: A8, LED_SMD:LED_0603_1608Metric_Pad1.05x0.95mm_HandSolder, F.Cu at (421.3, 150.5)
- added DS1: 7SEG, 8086PC:2181AS, F.Cu at (246.4, 105.1)
- added DS2: 7SEG, 8086PC:2181AS, F.Cu at (254.2, 105.1)
- added DS3: 7SEG, 8086PC:2181AS, F.Cu at (262.0, 105.1)
- added DS4: 7SEG, 8086PC:2181AS, F.Cu at (269.8, 105.1)
- added J2: RM68090, 8086PC:RM68090 RGB LCD module, F.Cu at (227.3, 71.7)
- added J3: RGB LCD, 8086PC:FPC_40, F.Cu at (222.5, 77.1)
- added J4: AVR-ISP-6, Connector_PinHeader_2.54mm:PinHeader_2x03_P2.54mm_Vertical, B.Cu at (518.8, 19.7)
- added J5: UART, Connector_PinHeader_2.54mm:PinHeader_1x04_P2.54mm_Vertical, B.Cu at (508.8, 27.1)
- added JP1: Write Protect, Jumper:SolderJumper-2_P1.3mm_Open_TrianglePad1.0x1.5mm, F.Cu at (314.2, 141.2)
- added JP2: LEDs, Jumper:SolderJumper-2_P1.3mm_Open_TrianglePad1.0x1.5mm, F.Cu at (314.2, 144.7)
- added JP3: MEM1, Jumper:SolderJumper-3_P2.0mm_Open_TrianglePad1.0x1.5mm, F.Cu at (315.5, 137.3)
- added JP4: Width, Jumper:SolderJumper-3_P2.0mm_Open_TrianglePad1.0x1.5mm, F.Cu at (352.2, 99.7)
- added JP5: LCD RST, Jumper:SolderJumper-3_P2.0mm_Open_TrianglePad1.0x1.5mm, F.Cu at (352.2, 105.7)
- added JP6: D/~{C}, Jumper:SolderJumper-3_P2.0mm_Open_TrianglePad1.0x1.5mm, F.Cu at (352.4, 111.7)
- added JP7: DISP, Jumper:SolderJumper-3_P2.0mm_Open_TrianglePad1.0x1.5mm, F.Cu at (352.2, 117.7)
- added R1: 5.11k, Resistor_SMD:R_0603_1608Metric_Pad0.98x0.95mm_HandSolder, F.Cu at (314.2, 46.7)
- added R10: 1k, Resistor_SMD:R_0603_1608Metric_Pad0.98x0.95mm_HandSolder, F.Cu at (481.8, 34.8)
- added R2: 5.11k, Resistor_SMD:R_0603_1608Metric_Pad0.98x0.95mm_HandSolder, F.Cu at (314.2, 49.2)
- added R3: 10k, Resistor_SMD:R_0603_1608Metric_Pad0.98x0.95mm_HandSolder, F.Cu at (314.2, 51.8)
- added R4: 22.1k, Resistor_SMD:R_0603_1608Metric_Pad0.98x0.95mm_HandSolder, F.Cu at (334.2, 56.4)
- added R5: 47.5k, Resistor_SMD:R_0603_1608Metric_Pad0.98x0.95mm_HandSolder, F.Cu at (334.2, 58.9)
- added R6: 100R, Resistor_SMD:R_0603_1608Metric_Pad0.98x0.95mm_HandSolder, F.Cu at (411.5, 54.7)
- added R7: 100R, Resistor_SMD:R_0603_1608Metric_Pad0.98x0.95mm_HandSolder, F.Cu at (411.5, 57.2)
- added R8: 100R, Resistor_SMD:R_0603_1608Metric_Pad0.98x0.95mm_HandSolder, F.Cu at (411.5, 59.8)
- added R9: 1k, Resistor_SMD:R_0603_1608Metric_Pad0.98x0.95mm_HandSolder, F.Cu at (481.8, 32.3)
- added TP1: ~{RTS}, TestPoint:TestPoint_Pad_1.5x1.5mm, F.Cu at (338.1, 59.1)
- added TP2: A, TestPoint:TestPoint_Pad_1.5x1.5mm, F.Cu at (379.4, 173.7)
- added TP3: B, TestPoint:TestPoint_Pad_1.5x1.5mm, F.Cu at (379.4, 177.3)
- added TP4: Y, TestPoint:TestPoint_Pad_1.5x1.5mm, F.Cu at (382.7, 177.5)
- added U27: 74AC373, Package_SO:SOIC-20W_7.5x12.8mm_P1.27mm, F.Cu at (324.9, 101.5)
- added U29: 74AC373, Package_SO:TSSOP-20_4.4x6.5mm_P0.65mm, F.Cu at (309.9, 112.7)
- added U38: 74HC165, Package_SO:SOIC-16_3.9x9.9mm_P1.27mm, F.Cu at (501.3, 20.3)
- added Y1: 16MHz, Crystal:Crystal_SMD_3225-4Pin_3.2x2.5mm_HandSoldering, F.Cu at (494.5, 28.8)
- BUS1: footprint Package_DIP:SMDIP-64_W15.24mm -> Connector_PinHeader_2.54mm:PinHeader_2x24_P2.54mm_Vertical
- RA1: value 220R -> 10k
- RA7: value 10k -> 220R
- SW1, SW10, SW11, SW12, SW13, SW14, SW15, SW16, SW17, SW18, SW19, SW2, SW20, SW21, SW22, SW23, SW24, SW25, SW26, SW27, SW28, SW29, SW3, SW30, SW31, SW32, SW4, SW5, SW6, SW7, SW8, SW9: footprint Button_Switch_SMD:SW_Push_1P1T_NO_6x6mm_H9.5mm -> 8086PC:SW_Push_1P1T_NO_6x6mm_H9.5mm
- SW33: value SW_Push -> RESET; footprint Button_Switch_SMD:SW_Push_1P1T_NO_6x6mm_H9.5mm -> 8086PC:SW_Push_1P1T_NO_6x6mm_H9.5mm
- U1: value 74HC02 -> P8086-2; footprint Package_SO:SOIC-14_3.9x8.7mm_P1.27mm -> Package_DIP:DIP-40_W15.24mm
- U10: value 74HC595 -> 74AC373; footprint Package_SO:SOIC-16W_7.5x10.3mm_P1.27mm -> Package_SO:SOIC-20W_7.5x12.8mm_P1.27mm
- U11, U12: value 74HC595 -> 74HC138; footprint Package_SO:SOIC-16W_7.5x10.3mm_P1.27mm -> Package_SO:SOIC-16_3.9x9.9mm_P1.27mm
- U13: value 74HC165 -> CXK58257AM; footprint Package_SO:SOIC-16W_7.5x10.3mm_P1.27mm -> Package_SO:SOIC-28W_7.5x17.9mm_P1.27mm
- U14: value 74HC165 -> IS61C256AH; footprint Package_SO:SOIC-16W_7.5x10.3mm_P1.27mm -> Package_SO:TSOP-I-28_11.8x8mm_P0.55mm
- U15: value AMS1117-3.3 -> IS61C256AH; footprint Package_TO_SOT_SMD:SOT-223-3_TabPin2 -> Package_SO:TSOP-I-28_11.8x8mm_P0.55mm
- U16: value 74AC373 -> IS61C256AH; footprint Package_SO:SOIC-20W_7.5x12.8mm_P1.27mm -> Package_SO:TSOP-I-28_11.8x8mm_P0.55mm
- U17: value CXK58257AM -> IS61C256AH; footprint Package_SO:SOIC-28W_7.5x17.9mm_P1.27mm -> Package_SO:TSOP-I-28_11.8x8mm_P0.55mm
- U18: value IS61C256AH -> IS61C3216; footprint Package_SO:TSOP-I-28_11.8x8mm_P0.55mm -> Package_SO:TSOP-II-44_10.16x18.41mm_P0.8mm
- U19: value IS61C256AH -> AM29F002; footprint Package_SO:TSOP-I-28_11.8x8mm_P0.55mm -> Package_SO:TSOP-I-32_18.4x8mm_P0.5mm
- U2: value ATmega328P-A -> 74AC00; footprint Package_QFP:TQFP-32_7x7mm_P0.8mm -> Package_SO:SOIC-14_3.9x8.7mm_P1.27mm
- U20: value IS61C3216 -> AM29F002; footprint Package_SO:TSOP-II-44_10.16x18.41mm_P0.8mm -> Package_SO:TSOP-I-32_18.4x8mm_P0.5mm
- U21: value IS61C256AH -> 28F400B5; footprint Package_SO:TSOP-I-28_11.8x8mm_P0.55mm -> Package_SO:TSOP-I-48_18.4x12mm_P0.5mm
- U22, U26: value AM29F002 -> 74AC373; footprint Package_SO:TSOP-I-32_18.4x8mm_P0.5mm -> Package_SO:SOIC-20W_7.5x12.8mm_P1.27mm
- U23: value 74HC14 -> 74AC373; footprint Package_SO:SOIC-14_3.9x8.7mm_P1.27mm -> Package_SO:SOIC-20W_7.5x12.8mm_P1.27mm
- U24: value 28F400B5 -> 74AC373; footprint Package_SO:TSOP-I-48_18.4x12mm_P0.5mm -> Package_SO:SOIC-20W_7.5x12.8mm_P1.27mm
- U25: value CP2102N-Axx-xQFN28 -> 74AC373; footprint Package_DFN_QFN:QFN-28-1EP_5x5mm_P0.5mm_EP3.35x3.35mm -> Package_SO:SOIC-20W_7.5x12.8mm_P1.27mm
- U3: value 74AC373 -> 74HC14; footprint Package_SO:SOIC-20W_7.5x12.8mm_P1.27mm -> Package_SO:SOIC-14_3.9x8.7mm_P1.27mm
- U30: value 74AC00 -> 74LVC245A; footprint Package_SO:SOIC-14_3.9x8.7mm_P1.27mm -> Package_SO:TSSOP-20_4.4x6.5mm_P0.65mm
- U31: value 74HC02 -> 74LVC245A; footprint Package_SO:SOIC-14_3.9x8.7mm_P1.27mm -> Package_SO:TSSOP-20_4.4x6.5mm_P0.65mm
- U32: value 74AC373 -> 74LVC245A; footprint Package_SO:SOIC-20W_7.5x12.8mm_P1.27mm -> Package_SO:TSSOP-20_4.4x6.5mm_P0.65mm
- U33: value 74AC373 -> ATmega328P; footprint Package_SO:SOIC-20W_7.5x12.8mm_P1.27mm -> Package_QFP:TQFP-32_7x7mm_P0.8mm
- U34, U35, U36: value 74AC373 -> 74HC595; footprint Package_SO:SOIC-20W_7.5x12.8mm_P1.27mm -> Package_SO:SOIC-16_3.9x9.9mm_P1.27mm
- U37: value 74AC373 -> 74HC165; footprint Package_SO:SOIC-20W_7.5x12.8mm_P1.27mm -> Package_SO:SOIC-16_3.9x9.9mm_P1.27mm
- U4, U5: value 74AC373 -> 74HC02; footprint Package_SO:SOIC-20W_7.5x12.8mm_P1.27mm -> Package_SO:SOIC-14_3.9x8.7mm_P1.27mm
- U6: value 74HC138 -> AMS1117-3.3; footprint Package_SO:SOIC-16_3.9x9.9mm_P1.27mm -> Package_TO_SOT_SMD:SOT-223-3_TabPin2
- U7: value 74HC138 -> CP2102N-Axx-xQFN28; footprint Package_SO:SOIC-16_3.9x9.9mm_P1.27mm -> Package_DFN_QFN:QFN-28-1EP_5x5mm_P0.5mm_EP3.35x3.35mm
- U8: value 74AC00 -> 74AC373; footprint Package_SO:SOIC-14_3.9x8.7mm_P1.27mm -> Package_SO:SOIC-20W_7.5x12.8mm_P1.27mm
- U9: value IS61C256AH -> 74AC373; footprint Package_SO:TSOP-I-28_11.8x8mm_P0.55mm -> Package_SO:SOIC-20W_7.5x12.8mm_P1.27mm
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Connections:
- BUS1 pad 10: AD9 -> ~{IO6}
- BUS1 pad 11: AD10 -> AD5
- BUS1 pad 12: AD11 -> ~{IO7}
- BUS1 pad 13: AD12 -> AD6
- BUS1 pad 14: AD13 -> ~{SEG2}
- BUS1 pad 15: AD14 -> AD7
- BUS1 pad 16: AD15 -> ~{SEG3}
- BUS1 pad 17: A16 -> AD8
- BUS1 pad 18: A17 -> ~{SEG4}
- BUS1 pad 19: A18 -> AD9
- BUS1 pad 2: AD1 -> ~{IO2}
- BUS1 pad 20: A19 -> ~{SEG5}
- BUS1 pad 21: ~{BHE} -> AD10
- BUS1 pad 22: BUSALE -> NMI
- BUS1 pad 23: ~{RD} -> AD11
- BUS1 pad 24: ~{WR} -> INTR
- BUS1 pad 25: ~{IO2} -> AD12
- BUS1 pad 26: ~{IO3} -> ~{INTA}
- BUS1 pad 27: ~{IO4} -> AD13
- BUS1 pad 28: ~{IO5} -> HOLD
- BUS1 pad 29: ~{IO6} -> AD14
- BUS1 pad 3: AD2 -> AD1
- BUS1 pad 30: ~{IO7} -> HLDA
- BUS1 pad 31: ~{SEG2} -> AD15
- BUS1 pad 32: ~{SEG3} -> ~{TEST}
- BUS1 pad 33: ~{SEG4} -> A16
- BUS1 pad 34: ~{SEG5} -> CLK
- BUS1 pad 35: NMI -> A17
- BUS1 pad 36: INTR -> RESET
- BUS1 pad 37: ~{INTA} -> A18
- BUS1 pad 38: HOLD -> READY
- BUS1 pad 39: HLDA -> A19
- BUS1 pad 4: AD3 -> ~{IO3}
- BUS1 pad 40: ~{TEST} -> +5V
- BUS1 pad 41: CLK -> ~{BHE}
- BUS1 pad 42: RESET -> +5V
- BUS1 pad 43: READY -> BUSALE
- BUS1 pad 44: +5V -> +3.3V
- BUS1 pad 45: +5V -> ~{RD}
- BUS1 pad 46: +3.3V -> GND
- BUS1 pad 47: GND -> ~{WR}
- BUS1 pad 5: AD4 -> AD2
- BUS1 pad 6: AD5 -> ~{IO4}
- BUS1 pad 7: AD6 -> AD3
- BUS1 pad 8: AD7 -> ~{IO5}
- BUS1 pad 9: AD8 -> AD4
- RA1 pad 1: /Memory/LA0 -> +5V
- RA1 pad 2: /Memory/LA1 -> +5V
- RA1 pad 3: /Memory/LA2 -> +5V
- RA1 pad 4: /Memory/LA3 -> GND
- RA1 pad 5: Net-(D51-A) -> RESET
- RA1 pad 6: Net-(D50-A) -> ~{RD}
- RA1 pad 7: Net-(D49-A) -> ~{WR}
- RA1 pad 8: Net-(D48-A) -> READY
- RA2 pad 1: /Memory/LA4 -> /Memory/LA0
- RA2 pad 2: /Memory/LA5 -> /Memory/LA1
- RA2 pad 3: /Memory/LA6 -> /Memory/LA2
- RA2 pad 4: /Memory/LA7 -> /Memory/LA3
- RA3 pad 1: /Memory/LA8 -> /Memory/LA4
- RA3 pad 2: /Memory/LA9 -> /Memory/LA5
- RA3 pad 3: /Memory/LA10 -> /Memory/LA6
- RA3 pad 4: /Memory/LA11 -> /Memory/LA7
- RA4 pad 1: /Memory/LA12 -> /Memory/LA8
- RA4 pad 2: /Memory/LA13 -> /Memory/LA9
- RA4 pad 3: /Memory/LA14 -> /Memory/LA10
- RA4 pad 4: /Memory/LA15 -> /Memory/LA11
- RA5 pad 1: /Memory/LA16 -> /Memory/LA12
- RA5 pad 2: /Memory/LA17 -> /Memory/LA13
- RA5 pad 3: /Memory/LA18 -> /Memory/LA14
- RA5 pad 4: /Memory/LA19 -> /Memory/LA15
- RA6 pad 1: +5V -> /Memory/LA16
- RA6 pad 2: /Memory/~{LBHE} -> /Memory/LA17
- RA6 pad 3: /Memory/SEG0 -> /Memory/LA18
- RA6 pad 4: /Memory/SEG1 -> /Memory/LA19
- RA7 pad 2: +5V -> /Memory/~{LBHE}
- RA7 pad 3: +5V -> /Memory/SEG0
- RA7 pad 4: GND -> /Memory/SEG1
- RA7 pad 5: RESET -> Net-(D24-A)
- RA7 pad 6: ~{RD} -> Net-(D23-A)
- RA7 pad 7: ~{WR} -> Net-(D22-A)
- RA7 pad 8: READY -> Net-(D21-A)
- U1 pad 1: Net-(U1-Pad1) -> GND
- U1 pad 10: unconnected-(U1-Pad10) -> AD6
- U1 pad 11: unconnected-(U1-Pad11) -> AD5
- U1 pad 12: unconnected-(U1-Pad12) -> AD4
- U1 pad 13: unconnected-(U1-Pad13) -> AD3
- U1 pad 14: +5V -> AD2
- U1 pad 2: /CPUALE -> AD14
- U1 pad 3: BUSALE -> AD13
- U1 pad 4: unconnected-(U1-Pad4) -> AD12
- U1 pad 5: unconnected-(U1-Pad5) -> AD11
- U1 pad 6: unconnected-(U1-Pad6) -> AD10
- U1 pad 7: GND -> AD9
- U1 pad 8: unconnected-(U1-Pad8) -> AD8
- U1 pad 9: unconnected-(U1-Pad9) -> AD7
- U10 pad 1: AD1 -> GND
- U10 pad 11: /Microcontroller/SPI_SCK -> ALE
- U10 pad 12: /Microcontroller/REG_RCLK -> /Memory/~{LBHE}
- U10 pad 13: /Microcontroller/REG_OE -> ~{BHE}
- U10 pad 14: /Microcontroller/SPI_MOSI -> unconnected-(U10-D5-Pad14)
- U10 pad 15: AD0 -> unconnected-(U10-O5-Pad15)
- U10 pad 16: +5V -> unconnected-(U10-O6-Pad16)
- U10 pad 2: AD2 -> /Memory/LA16
- U10 pad 3: AD3 -> A16
- U10 pad 4: AD4 -> A17
- U10 pad 5: AD5 -> /Memory/LA17
- U10 pad 6: AD6 -> /Memory/LA18
- U10 pad 7: AD7 -> A18
- U10 pad 8: GND -> A19
- U10 pad 9: Net-(U10-QH') -> /Memory/LA19
- U11 pad 1: AD9 -> /Memory/LA16
- U11 pad 10: GND -> ~{SEG5}
- U11 pad 11: /Microcontroller/SPI_SCK -> ~{SEG4}
- U11 pad 12: /Microcontroller/REG_RCLK -> ~{SEG3}
- U11 pad 13: /Microcontroller/REG_OE -> ~{SEG2}
- U11 pad 14: Net-(U10-QH') -> ~{SEG1}
- U11 pad 15: AD8 -> ~{SEG0}
- U11 pad 2: AD10 -> /Memory/LA17
- U11 pad 3: AD11 -> /Memory/LA18
- U11 pad 4: AD12 -> /Memory/LA19
- U11 pad 5: AD13 -> /Memory/LA19
- U11 pad 6: AD14 -> M\~{IO}
- U11 pad 7: AD15 -> ~{SEG7}
- U11 pad 9: Net-(U11-QH') -> ~{SEG6}
- U12 pad 1: A17 -> /Memory/LA1
- U12 pad 10: GND -> ~{IO5}
- U12 pad 11: /Microcontroller/SPI_SCK -> ~{IO4}
- U12 pad 12: /Microcontroller/REG_RCLK -> ~{IO3}
- U12 pad 13: /Microcontroller/REG_OE -> ~{IO2}
- U12 pad 14: Net-(U11-QH') -> ~{IO1}
- U12 pad 15: A16 -> ~{IO0}
- U12 pad 2: A18 -> /Memory/LA2
- U12 pad 3: A19 -> /Memory/LA3
- U12 pad 4: unconnected-(U12-QE-Pad4) -> M\~{IO}
- U12 pad 5: unconnected-(U12-QF-Pad5) -> M\~{IO}
- U12 pad 6: unconnected-(U12-QG-Pad6) -> +5V
- U12 pad 7: unconnected-(U12-QH-Pad7) -> ~{IO7}
- U12 pad 9: unconnected-(U12-QH'-Pad9) -> ~{IO6}
- U13 pad 1: /Microcontroller/REG_SHLD -> /Memory/LA15
- U13 pad 10: unconnected-(U13-SER-Pad10) -> /Memory/LA1
- U13 pad 14: AD3 -> GND
- U13 pad 15: unconnected-(U13-~{CE}-Pad15) -> AD3
- U13 pad 16: +5V -> AD4
- U13 pad 2: unconnected-(U13-CLK-Pad2) -> /Memory/LA13
- U13 pad 3: AD4 -> /Memory/LA8
- U13 pad 4: AD5 -> /Memory/LA7
- U13 pad 5: AD6 -> /Memory/LA6
- U13 pad 6: AD7 -> /Memory/LA5
- U13 pad 7: unconnected-(U13-~{QH}-Pad7) -> /Memory/LA4
- U13 pad 8: GND -> /Memory/LA3
- U13 pad 9: unconnected-(U13-QH-Pad9) -> /Memory/LA2
- U14 pad 1: /Microcontroller/REG_SHLD -> /Memory/LA15
- U14 pad 10: unconnected-(U14-SER-Pad10) -> /Memory/LA1
- U14 pad 11: AD8 -> AD0
- U14 pad 12: AD9 -> AD1
- U14 pad 13: AD10 -> AD2
- U14 pad 14: AD11 -> GND
- U14 pad 15: unconnected-(U14-~{CE}-Pad15) -> AD3
- U14 pad 16: +5V -> AD4
- U14 pad 2: unconnected-(U14-CLK-Pad2) -> /Memory/LA13
- U14 pad 3: AD12 -> /Memory/LA8
- U14 pad 4: AD13 -> /Memory/LA7
- U14 pad 5: AD14 -> /Memory/LA6
- U14 pad 6: AD15 -> /Memory/LA5
- U14 pad 7: unconnected-(U14-~{QH}-Pad7) -> /Memory/LA4
- U14 pad 8: GND -> /Memory/LA3
- U14 pad 9: /Microcontroller/SPI_MISO -> /Memory/LA2
- U15 pad 1: GND -> /Memory/LA15
- U15 pad 2: +3.3V -> /Memory/LA13
- U15 pad 3: +5V -> /Memory/LA8
- U16 pad 1: /IO/~{RD0} -> /Memory/LA15
- U16 pad 10: GND -> /Memory/LA1
- U16 pad 11: +5V -> AD0
- U16 pad 12: AD4 -> AD1
- U16 pad 13: /IO/I4 -> AD2
- U16 pad 14: /IO/I5 -> GND
- U16 pad 15: AD5 -> AD3
- U16 pad 16: AD6 -> AD4
- U16 pad 17: /IO/I6 -> AD5
- U16 pad 18: /IO/I7 -> AD6
- U16 pad 2: AD0 -> /Memory/LA13
- U16 pad 20: +5V -> /Memory/~{MEM1L}
- U16 pad 3: /IO/I0 -> /Memory/LA8
- U16 pad 4: /IO/I1 -> /Memory/LA7
- U16 pad 5: AD1 -> /Memory/LA6
- U16 pad 6: AD2 -> /Memory/LA5
- U16 pad 7: /IO/I2 -> /Memory/LA4
- U16 pad 8: /IO/I3 -> /Memory/LA3
- U16 pad 9: AD3 -> /Memory/LA2
- U17 pad 11: AD0 -> AD8
- U17 pad 12: AD1 -> AD9
- U17 pad 13: AD2 -> AD10
- U17 pad 15: AD3 -> AD11
- U17 pad 16: AD4 -> AD12
- U17 pad 17: AD5 -> AD13
- U17 pad 18: AD6 -> AD14
- U17 pad 19: AD7 -> AD15
- U17 pad 20: /Memory/~{SEG0L} -> /Memory/~{MEM1H}
- U18 pad 1: /Memory/LA15 -> unconnected-(U18-NC-Pad1)
- U18 pad 10: /Memory/LA1 -> AD3
- U18 pad 11: AD8 -> +5V
- U18 pad 12: AD9 -> GND
- U18 pad 13: AD10 -> AD4
- U18 pad 14: GND -> AD5
- U18 pad 15: AD11 -> AD6
- U18 pad 16: AD12 -> AD7
- U18 pad 17: AD13 -> ~{WR}
- U18 pad 18: AD14 -> /Memory/LA11
- U18 pad 19: AD15 -> /Memory/LA10
- U18 pad 2: /Memory/LA13 -> /Memory/LA15
- U18 pad 20: /Memory/~{SEG0H} -> /Memory/LA9
- U18 pad 21: /Memory/LA11 -> /Memory/LA8
- U18 pad 22: ~{WR} -> unconnected-(U18-NC-Pad22)
- U18 pad 23: /Memory/LA12 -> unconnected-(U18-NC-Pad23)
- U18 pad 24: /Memory/LA10 -> /Memory/LA7
- U18 pad 25: /Memory/LA9 -> /Memory/LA6
- U18 pad 26: /Memory/LA14 -> /Memory/LA5
- U18 pad 27: ~{RD} -> /Memory/LA4
- U18 pad 28: +5V -> unconnected-(U18-NC-Pad28)
- U18 pad 3: /Memory/LA8 -> /Memory/LA14
- U18 pad 4: /Memory/LA7 -> /Memory/LA13
- U18 pad 5: /Memory/LA6 -> /Memory/LA12
- U18 pad 6: /Memory/LA5 -> ~{SEG1}
- U18 pad 7: /Memory/LA4 -> AD0
- U18 pad 8: /Memory/LA3 -> AD1
- U18 pad 9: /Memory/LA2 -> AD2
- U19 pad 1: /Memory/LA15 -> /Memory/LA12
- U19 pad 10: /Memory/LA1 -> /Memory/LA17
- U19 pad 11: AD0 -> /Memory/LA16
- U19 pad 12: AD1 -> /Memory/LA13
- U19 pad 13: AD2 -> /Memory/LA8
- U19 pad 14: GND -> /Memory/LA7
- U19 pad 15: AD3 -> /Memory/LA6
- U19 pad 16: AD4 -> /Memory/LA5
- U19 pad 17: AD5 -> /Memory/LA4
- U19 pad 18: AD6 -> /Memory/LA3
- U19 pad 19: AD7 -> /Memory/LA2
- U19 pad 2: /Memory/LA13 -> /Memory/LA10
- U19 pad 20: /Memory/~{MEM1L} -> /Memory/LA1
- U19 pad 21: /Memory/LA11 -> AD0
- U19 pad 22: ~{RD} -> AD1
- U19 pad 23: /Memory/LA12 -> AD2
- U19 pad 24: /Memory/LA10 -> GND
- U19 pad 25: /Memory/LA9 -> AD3
- U19 pad 26: /Memory/LA14 -> AD4
- U19 pad 27: ~{WR} -> AD5
- U19 pad 28: +5V -> AD6
- U19 pad 3: /Memory/LA8 -> /Memory/LA9
- U19 pad 4: /Memory/LA7 -> /Memory/LA14
- U19 pad 5: /Memory/LA6 -> /Memory/LA15
- U19 pad 6: /Memory/LA5 -> /Memory/LA18
- U19 pad 7: /Memory/LA4 -> /Memory/~{WRP}
- U19 pad 8: /Memory/LA3 -> +5V
- U19 pad 9: /Memory/LA2 -> +5V
- U2 pad 1: ~{WR} -> /Memory/~{LA0}
- U2 pad 10: Net-(U2-PD6) -> /Memory/MEM1
- U2 pad 11: ~{INTA} -> /Memory/~{MEM1H}
- U2 pad 12: HOLD -> /Memory/MEM1
- U2 pad 13: HLDA -> /Memory/LBHE
- U2 pad 14: /Microcontroller/REG_RCLK -> +5V
- U2 pad 2: BUSALE -> /Memory/SEG0
- U2 pad 3: GND -> /Memory/~{SEG0L}
- U2 pad 4: +5V -> /Memory/SEG0
- U2 pad 5: GND -> /Memory/LBHE
- U2 pad 6: +5V -> /Memory/~{SEG0H}
- U2 pad 7: unconnected-(U2-XTAL1/PB6-Pad7) -> GND
- U2 pad 8: unconnected-(U2-XTAL2/PB7-Pad8) -> /Memory/~{MEM1L}
- U2 pad 9: CLK -> /Memory/~{LA0}
- U20 pad 1: unconnected-(U20-NC-Pad1) -> /Memory/LA12
- U20 pad 10: AD3 -> /Memory/LA17
- U20 pad 11: +5V -> /Memory/LA16
- U20 pad 12: GND -> /Memory/LA13
- U20 pad 13: AD4 -> /Memory/LA8
- U20 pad 14: AD5 -> /Memory/LA7
- U20 pad 15: AD6 -> /Memory/LA6
- U20 pad 16: AD7 -> /Memory/LA5
- U20 pad 17: ~{WR} -> /Memory/LA4
- U20 pad 18: /Memory/LA11 -> /Memory/LA3
- U20 pad 19: /Memory/LA10 -> /Memory/LA2
- U20 pad 2: /Memory/LA15 -> /Memory/LA10
- U20 pad 20: /Memory/LA9 -> /Memory/LA1
- U20 pad 21: /Memory/LA8 -> AD8
- U20 pad 22: unconnected-(U20-NC-Pad22) -> AD9
- U20 pad 23: unconnected-(U20-NC-Pad23) -> AD10
- U20 pad 24: /Memory/LA7 -> GND
- U20 pad 25: /Memory/LA6 -> AD11
- U20 pad 26: /Memory/LA5 -> AD12
- U20 pad 27: /Memory/LA4 -> AD13
- U20 pad 28: unconnected-(U20-NC-Pad28) -> AD14
- U20 pad 29: AD8 -> AD15
- U20 pad 3: /Memory/LA14 -> /Memory/LA9
- U20 pad 30: AD9 -> /Memory/~{MEM1H}
- U20 pad 31: AD10 -> /Memory/LA11
- U20 pad 32: AD11 -> ~{RD}
- U20 pad 4: /Memory/LA13 -> /Memory/LA14
- U20 pad 5: /Memory/LA12 -> /Memory/LA15
- U20 pad 6: ~{SEG1} -> /Memory/LA18
- U20 pad 7: AD0 -> /Memory/~{WRP}
- U20 pad 8: AD1 -> +5V
- U20 pad 9: AD2 -> +5V
- U21 pad 1: /Memory/LA15 -> /Memory/LA16
- U21 pad 10: /Memory/LA1 -> unconnected-(U21-NC-Pad10)
- U21 pad 11: AD8 -> /Memory/~{WRP}
- U21 pad 12: AD9 -> +5V
- U21 pad 13: AD10 -> +5V
- U21 pad 14: GND -> +5V
- U21 pad 15: AD11 -> unconnected-(U21-NC-Pad15)
- U21 pad 16: AD12 -> unconnected-(U21-NC-Pad16)
- U21 pad 17: AD13 -> /Memory/LA18
- U21 pad 18: AD14 -> /Memory/LA8
- U21 pad 19: AD15 -> /Memory/LA7
- U21 pad 2: /Memory/LA13 -> /Memory/LA15
- U21 pad 20: /Memory/~{MEM1H} -> /Memory/LA6
- U21 pad 21: /Memory/LA11 -> /Memory/LA5
- U21 pad 22: ~{RD} -> /Memory/LA4
- U21 pad 23: /Memory/LA12 -> /Memory/LA3
- U21 pad 24: /Memory/LA10 -> /Memory/LA2
- U21 pad 25: /Memory/LA9 -> /Memory/LA1
- U21 pad 26: /Memory/LA14 -> /Memory/~{LA19}
- U21 pad 27: ~{WR} -> GND
- U21 pad 28: +5V -> ~{RD}
- U21 pad 3: /Memory/LA8 -> /Memory/LA14
- U21 pad 4: /Memory/LA7 -> /Memory/LA13
- U21 pad 5: /Memory/LA6 -> /Memory/LA12
- U21 pad 6: /Memory/LA5 -> /Memory/LA11
- U21 pad 7: /Memory/LA4 -> /Memory/LA10
- U21 pad 8: /Memory/LA3 -> /Memory/LA9
- U21 pad 9: /Memory/LA2 -> unconnected-(U21-NC-Pad9)
- U22 pad 1: /Memory/LA12 -> GND
- U22 pad 10: /Memory/LA17 -> GND
- U22 pad 11: /Memory/LA16 -> /IO/WR0
- U22 pad 12: /Memory/LA13 -> /IO/O4
- U22 pad 13: /Memory/LA8 -> AD4
- U22 pad 14: /Memory/LA7 -> AD5
- U22 pad 15: /Memory/LA6 -> /IO/O5
- U22 pad 16: /Memory/LA5 -> /IO/O6
- U22 pad 17: /Memory/LA4 -> AD6
- U22 pad 18: /Memory/LA3 -> AD7
- U22 pad 19: /Memory/LA2 -> /IO/O7
- U22 pad 2: /Memory/LA10 -> /IO/O0
- U22 pad 20: /Memory/LA1 -> +5V
- U22 pad 3: /Memory/LA9 -> AD0
- U22 pad 4: /Memory/LA14 -> AD1
- U22 pad 5: /Memory/LA15 -> /IO/O1
- U22 pad 6: /Memory/LA18 -> /IO/O2
- U22 pad 7: /Memory/~{WRP} -> AD2
- U22 pad 8: +5V -> AD3
- U22 pad 9: +5V -> /IO/O3
- U23 pad 1: /Memory/LA0 -> GND
- U23 pad 10: /Memory/LBHE -> GND
- U23 pad 11: /Memory/~{LBHE} -> /IO/WR0
- U23 pad 12: ALE -> /IO/O12
- U23 pad 13: Net-(U1-Pad1) -> AD12
- U23 pad 14: +5V -> AD13
- U23 pad 2: /Memory/~{LA0} -> /IO/O8
- U23 pad 3: /Memory/LA19 -> AD8
- U23 pad 4: /Memory/~{LA19} -> AD9
- U23 pad 5: ~{SEG1} -> /IO/O9
- U23 pad 6: /Memory/SEG1 -> /IO/O10
- U23 pad 7: GND -> AD10
- U23 pad 8: /Memory/SEG0 -> AD11
- U23 pad 9: ~{SEG0} -> /IO/O11
- U24 pad 1: /Memory/LA16 -> GND
- U24 pad 10: unconnected-(U24-NC-Pad10) -> GND
- U24 pad 11: /Memory/~{WRP} -> /IO/WR1
- U24 pad 12: +5V -> /IO/O20
- U24 pad 13: +5V -> AD4
- U24 pad 14: +5V -> AD5
- U24 pad 15: unconnected-(U24-NC-Pad15) -> /IO/O21
- U24 pad 16: unconnected-(U24-NC-Pad16) -> /IO/O22
- U24 pad 17: /Memory/LA18 -> AD6
- U24 pad 18: /Memory/LA8 -> AD7
- U24 pad 19: /Memory/LA7 -> /IO/O23
- U24 pad 2: /Memory/LA15 -> /IO/O16
- U24 pad 20: /Memory/LA6 -> +5V
- U24 pad 3: /Memory/LA14 -> AD0
- U24 pad 4: /Memory/LA13 -> AD1
- U24 pad 5: /Memory/LA12 -> /IO/O17
- U24 pad 6: /Memory/LA11 -> /IO/O18
- U24 pad 7: /Memory/LA10 -> AD2
- U24 pad 8: /Memory/LA9 -> AD3
- U24 pad 9: unconnected-(U24-NC-Pad9) -> /IO/O19
- U25 pad 1: unconnected-(U25-~{DCD}-Pad1) -> GND
- U25 pad 10: unconnected-(U25-NC-Pad10) -> GND
- U25 pad 11: unconnected-(U25-~{SUSPEND}-Pad11) -> /IO/WR1
- U25 pad 12: unconnected-(U25-SUSPEND-Pad12) -> /IO/O28
- U25 pad 13: unconnected-(U25-CHREN-Pad13) -> AD12
- U25 pad 14: unconnected-(U25-CHR1-Pad14) -> AD13
- U25 pad 15: unconnected-(U25-CHR0-Pad15) -> /IO/O29
- U25 pad 16: unconnected-(U25-~{WAKEUP}/GPIO.3-Pad16) -> /IO/O30
- U25 pad 17: unconnected-(U25-RS485/GPIO.2-Pad17) -> AD14
- U25 pad 18: unconnected-(U25-~{RXT}/GPIO.1-Pad18) -> AD15
- U25 pad 19: unconnected-(U25-~{TXT}/GPIO.0-Pad19) -> /IO/O31
- U25 pad 2: unconnected-(U25-~{RI}/CLK-Pad2) -> /IO/O24
- U25 pad 20: unconnected-(U25-GPIO.6-Pad20) -> +5V
- U25 pad 3: unconnected-(U25-GND-Pad29) -> AD8
- U25 pad 4: unconnected-(U25-D+-Pad4) -> AD9
- U25 pad 5: unconnected-(U25-D--Pad5) -> /IO/O25
- U25 pad 6: unconnected-(U25-VDD-Pad6) -> /IO/O26
- U25 pad 7: unconnected-(U25-VREGIN-Pad7) -> AD10
- U25 pad 8: unconnected-(U25-VBUS-Pad8) -> AD11
- U25 pad 9: unconnected-(U25-~{RST}-Pad9) -> /IO/O27
- U26 pad 1: /Memory/LA12 -> /IO/~{RD0}
- U26 pad 10: /Memory/LA17 -> GND
- U26 pad 11: /Memory/LA16 -> +5V
- U26 pad 12: /Memory/LA13 -> AD4
- U26 pad 13: /Memory/LA8 -> /IO/I4
- U26 pad 14: /Memory/LA7 -> /IO/I5
- U26 pad 15: /Memory/LA6 -> AD5
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Routing:
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Other:
- board text removed: "7 segment"
- board text removed: "RGB LCD"

Commit message: start memory layout
Parts:
- removed the U14 at (446.0, 63.6)
- removed the U15 at (455.7, 63.6)
- added U1: P8086-2, Package_DIP:DIP-40_W15.24mm, B.Cu at (-235.3, 147.7)
- added U10: 74AC573, Package_SO:TSSOP-20_4.4x6.5mm_P0.65mm, B.Cu at (-242.4, 150.3)
- added U13: CXK58257AM, Package_SO:SOIC-28W_7.5x17.9mm_P1.27mm, F.Cu at (-103.8, 35.2)
- added U13: CXK58257AM, Package_SO:SOIC-28W_7.5x17.9mm_P1.27mm, B.Cu at (-67.3, 107.7)
- added U14: IS61C256AH, Package_SO:TSOP-I-28_11.8x8mm_P0.55mm, F.Cu at (-109.0, 34.9)
- added U14: IS61C256AH, Package_SO:TSOP-I-28_11.8x8mm_P0.55mm, B.Cu at (-72.6, 107.7)
- added U14: IS61C256AH, Package_SO:TSOP-I-28_11.8x8mm_P0.55mm, B.Cu at (-32.8, 76.0)
- added U15: IS61C256AH, Package_SO:TSOP-I-28_11.8x8mm_P0.55mm, B.Cu at (-51.6, 76.0)
- added U15: IS61C256AH, Package_SO:TSOP-I-28_11.8x8mm_P0.55mm, B.Cu at (-109.0, 34.9)
- added U15: IS61C256AH, Package_SO:TSOP-I-28_11.8x8mm_P0.55mm, B.Cu at (-91.6, 107.7)
- added U16: IS61C256AH, Package_SO:TSOP-I-28_11.8x8mm_P0.55mm, F.Cu at (-126.3, 34.9)
- added U16: IS61C256AH, Package_SO:TSOP-I-28_11.8x8mm_P0.55mm, B.Cu at (-110.6, 107.7)
- added U17: IS61C256AH, Package_SO:TSOP-I-28_11.8x8mm_P0.55mm, B.Cu at (-129.6, 107.7)
- added U17: IS61C256AH, Package_SO:TSOP-I-28_11.8x8mm_P0.55mm, B.Cu at (-126.3, 34.9)
- added U8: 74AC573, Package_SO:TSSOP-20_4.4x6.5mm_P0.65mm, B.Cu at (-224.9, 139.2)
- added U9: 74AC573, Package_SO:TSSOP-20_4.4x6.5mm_P0.65mm, B.Cu at (-233.3, 139.2)
- DS1, DS2, DS3, DS4, JP1, JP2, JP3: moved to B.Cu
- U10, U22, U23, U24, U25, U26, U27, U28, U8, U9: value 74AC373 -> 74AC573; footprint Package_SO:SOIC-20W_7.5x12.8mm_P1.27mm -> Package_SO:TSSOP-20_4.4x6.5mm_P0.65mm
- U17: renamed from U16; moved to B.Cu
- U29: value 74AC373 -> 74AC573
- moved U18 566.0 mm to (-87.1, 65.4)
- moved U17 545.6 mm to (-51.6, 61.4)
- moved U1 535.2 mm to (-131.5, 141.2)
- moved U16 526.9 mm to (-32.8, 61.4)
- moved U10 479.6 mm to (-138.4, 153.9)
- moved U13 478.4 mm to (-27.6, 76.0), turned to 0 degrees
- moved U9 477.4 mm to (-122.6, 135.1), turned to 90 degrees
- moved U8 443.4 mm to (-102.3, 135.1)
- moved U19 306.0 mm to (150.7, 101.5)
- moved U20 306.0 mm to (150.7, 111.0)
- moved U21 306.0 mm to (150.7, 122.6)
- moved RA1 272.6 mm to (127.2, 38.9)
- moved SW33 272.6 mm to (119.3, 40.6)
- moved JP3 256.7 mm to (83.3, 27.9), turned to 180 degrees
- moved JP1 254.3 mm to (84.6, 31.8), turned to 180 degrees
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- renumbered SW8 to SW5, SW5 to SW8, U17 to U16
Connections:
- SW5 pad 2: /IO/I7 -> /IO/I4
- SW8 pad 2: /IO/I4 -> /IO/I7
- U10 pad 12: /Memory/~{LBHE} -> unconnected-(U10-O7-Pad12)
- U10 pad 13: ~{BHE} -> unconnected-(U10-O6-Pad13)
- U10 pad 15: unconnected-(U10-O5-Pad15) -> /Memory/~{LBHE}
- U10 pad 16: unconnected-(U10-O6-Pad16) -> /Memory/LA19
- U10 pad 17: unconnected-(U10-D6-Pad17) -> /Memory/LA18
- U10 pad 18: unconnected-(U10-D7-Pad18) -> /Memory/LA17
- U10 pad 19: unconnected-(U10-O7-Pad19) -> /Memory/LA16
- U10 pad 2: /Memory/LA16 -> A16
- U10 pad 3: A16 -> A17
- U10 pad 4: A17 -> A18
- U10 pad 5: /Memory/LA17 -> A19
- U10 pad 6: /Memory/LA18 -> ~{BHE}
- U10 pad 7: A18 -> GND
- U10 pad 8: A19 -> GND
- U10 pad 9: /Memory/LA19 -> GND
- U16 pad 11: AD8 -> AD0
- U16 pad 12: AD9 -> AD1
- U16 pad 13: AD10 -> AD2
- U16 pad 15: AD11 -> AD3
- U16 pad 16: AD12 -> AD4
- U16 pad 17: AD13 -> AD5
- U16 pad 18: AD14 -> AD6
- U16 pad 19: AD15 -> AD7
- U16 pad 20: /Memory/~{MEM1H} -> /Memory/~{MEM1L}
- U17 pad 11: AD0 -> AD8
- U17 pad 12: AD1 -> AD9
- U17 pad 13: AD2 -> AD10
- U17 pad 15: AD3 -> AD11
- U17 pad 16: AD4 -> AD12
- U17 pad 17: AD5 -> AD13
- U17 pad 18: AD6 -> AD14
- U17 pad 19: AD7 -> AD15
- U17 pad 20: /Memory/~{MEM1L} -> /Memory/~{MEM1H}
- U22 pad 12: /IO/O4 -> /IO/O7
- U22 pad 13: AD4 -> /IO/O6
- U22 pad 14: AD5 -> /IO/O5
- U22 pad 15: /IO/O5 -> /IO/O4
- U22 pad 16: /IO/O6 -> /IO/O3
- U22 pad 17: AD6 -> /IO/O2
- U22 pad 18: AD7 -> /IO/O1
- U22 pad 19: /IO/O7 -> /IO/O0
- U22 pad 2: /IO/O0 -> AD0
- U22 pad 3: AD0 -> AD1
- U22 pad 4: AD1 -> AD2
- U22 pad 5: /IO/O1 -> AD3
- U22 pad 6: /IO/O2 -> AD4
- U22 pad 7: AD2 -> AD5
- U22 pad 8: AD3 -> AD6
- U22 pad 9: /IO/O3 -> AD7
- U23 pad 12: /IO/O12 -> /IO/O15
- U23 pad 13: AD12 -> /IO/O14
- U23 pad 14: AD13 -> /IO/O13
- U23 pad 15: /IO/O13 -> /IO/O12
- U23 pad 16: /IO/O14 -> /IO/O11
- U23 pad 17: AD14 -> /IO/O10
- U23 pad 18: AD15 -> /IO/O9
- U23 pad 19: /IO/O15 -> /IO/O8
- U23 pad 2: /IO/O8 -> AD8
- U23 pad 3: AD8 -> AD9
- U23 pad 4: AD9 -> AD10
- U23 pad 5: /IO/O9 -> AD11
- U23 pad 6: /IO/O10 -> AD12
- U23 pad 7: AD10 -> AD13
- U23 pad 8: AD11 -> AD14
- U23 pad 9: /IO/O11 -> AD15
- U24 pad 12: /IO/O20 -> /IO/O23
- U24 pad 13: AD4 -> /IO/O22
- U24 pad 14: AD5 -> /IO/O21
- U24 pad 15: /IO/O21 -> /IO/O20
- U24 pad 16: /IO/O22 -> /IO/O19
- U24 pad 17: AD6 -> /IO/O18
- U24 pad 18: AD7 -> /IO/O17
- U24 pad 19: /IO/O23 -> /IO/O16
- U24 pad 2: /IO/O16 -> AD0
- U24 pad 3: AD0 -> AD1
- U24 pad 4: AD1 -> AD2
- U24 pad 5: /IO/O17 -> AD3
- U24 pad 6: /IO/O18 -> AD4
- U24 pad 7: AD2 -> AD5
- U24 pad 8: AD3 -> AD6
- U24 pad 9: /IO/O19 -> AD7
- U25 pad 12: /IO/O28 -> /IO/O31
- U25 pad 13: AD12 -> /IO/O30
- U25 pad 14: AD13 -> /IO/O29
- U25 pad 15: /IO/O29 -> /IO/O28
- U25 pad 16: /IO/O30 -> /IO/O27
- U25 pad 17: AD14 -> /IO/O26
- U25 pad 18: AD15 -> /IO/O25
- U25 pad 19: /IO/O31 -> /IO/O24
- U25 pad 2: /IO/O24 -> AD8
- U25 pad 3: AD8 -> AD9
- U25 pad 4: AD9 -> AD10
- U25 pad 5: /IO/O25 -> AD11
- U25 pad 6: /IO/O26 -> AD12
- U25 pad 7: AD10 -> AD13
- U25 pad 8: AD11 -> AD14
- U25 pad 9: /IO/O27 -> AD15
- U26 pad 12: AD4 -> AD7
- U26 pad 13: /IO/I4 -> AD6
- U26 pad 14: /IO/I5 -> AD5
- U26 pad 15: AD5 -> AD4
- U26 pad 16: AD6 -> AD3
- U26 pad 17: /IO/I6 -> AD2
- U26 pad 18: /IO/I7 -> AD1
- U26 pad 19: AD7 -> AD0
- U26 pad 2: AD0 -> /IO/I0
- U26 pad 3: /IO/I0 -> /IO/I1
- U26 pad 4: /IO/I1 -> /IO/I2
- U26 pad 5: AD1 -> /IO/I3
- U26 pad 6: AD2 -> /IO/I4
- U26 pad 7: /IO/I2 -> /IO/I5
- U26 pad 8: /IO/I3 -> /IO/I6
- U26 pad 9: AD3 -> /IO/I7
- U27 pad 12: AD12 -> AD15
- U27 pad 13: /IO/I12 -> AD14
- U27 pad 14: /IO/I13 -> AD13
- U27 pad 15: AD13 -> AD12
- U27 pad 16: AD14 -> AD11
- U27 pad 17: /IO/I14 -> AD10
- U27 pad 18: /IO/I15 -> AD9
- U27 pad 19: AD15 -> AD8
- U27 pad 2: AD8 -> /IO/I8
- U27 pad 3: /IO/I8 -> /IO/I9
- U27 pad 4: /IO/I9 -> /IO/I10
- U27 pad 5: AD9 -> /IO/I11
- U27 pad 6: AD10 -> /IO/I12
- U27 pad 7: /IO/I10 -> /IO/I13
- U27 pad 8: /IO/I11 -> /IO/I14
- U27 pad 9: AD11 -> /IO/I15
- U28 pad 12: AD4 -> AD7
- U28 pad 13: /IO/I20 -> AD6
- U28 pad 14: /IO/I21 -> AD5
- U28 pad 15: AD5 -> AD4
- U28 pad 16: AD6 -> AD3
- U28 pad 17: /IO/I22 -> AD2
- U28 pad 18: /IO/I23 -> AD1
- U28 pad 19: AD7 -> AD0
- U28 pad 2: AD0 -> /IO/I16
- U28 pad 3: /IO/I16 -> /IO/I17
- U28 pad 4: /IO/I17 -> /IO/I18
- U28 pad 5: AD1 -> /IO/I19
- U28 pad 6: AD2 -> /IO/I20
- U28 pad 7: /IO/I18 -> /IO/I21
- U28 pad 8: /IO/I19 -> /IO/I22
- U28 pad 9: AD3 -> /IO/I23
- U29 pad 12: AD12 -> AD15
- U29 pad 13: /IO/I28 -> AD14
- U29 pad 14: /IO/I29 -> AD13
- U29 pad 15: AD13 -> AD12
- U29 pad 16: AD14 -> AD11
- U29 pad 17: /IO/I30 -> AD10
- U29 pad 18: /IO/I31 -> AD9
- U29 pad 19: AD15 -> AD8
- U29 pad 2: AD8 -> /IO/I24
- U29 pad 3: /IO/I24 -> /IO/I25
- U29 pad 4: /IO/I25 -> /IO/I26
- U29 pad 5: AD9 -> /IO/I27
- U29 pad 6: AD10 -> /IO/I28
- U29 pad 7: /IO/I26 -> /IO/I29
- U29 pad 8: /IO/I27 -> /IO/I30
- U29 pad 9: AD11 -> /IO/I31
- U8 pad 12: /Memory/LA4 -> /Memory/LA7
- U8 pad 13: AD4 -> /Memory/LA6
- U8 pad 14: AD5 -> /Memory/LA5
- U8 pad 15: /Memory/LA5 -> /Memory/LA4
- U8 pad 16: /Memory/LA6 -> /Memory/LA3
- U8 pad 17: AD6 -> /Memory/LA2
- U8 pad 18: AD7 -> /Memory/LA1
- U8 pad 19: /Memory/LA7 -> /Memory/LA0
- U8 pad 2: /Memory/LA0 -> AD0
- U8 pad 3: AD0 -> AD1
- U8 pad 4: AD1 -> AD2
- U8 pad 5: /Memory/LA1 -> AD3
- U8 pad 6: /Memory/LA2 -> AD4
- U8 pad 7: AD2 -> AD5
- U8 pad 8: AD3 -> AD6
- U8 pad 9: /Memory/LA3 -> AD7
- U9 pad 12: /Memory/LA12 -> /Memory/LA15
- U9 pad 13: AD12 -> /Memory/LA14
- U9 pad 14: AD13 -> /Memory/LA13
- U9 pad 15: /Memory/LA13 -> /Memory/LA12
- U9 pad 16: /Memory/LA14 -> /Memory/LA11
- U9 pad 17: AD14 -> /Memory/LA10
- U9 pad 18: AD15 -> /Memory/LA9
- U9 pad 19: /Memory/LA15 -> /Memory/LA8
- U9 pad 2: /Memory/LA8 -> AD8
- U9 pad 3: AD8 -> AD9
- U9 pad 4: AD9 -> AD10
- U9 pad 5: /Memory/LA9 -> AD11
- U9 pad 6: /Memory/LA10 -> AD12
- U9 pad 7: AD10 -> AD13
- U9 pad 8: AD11 -> AD14
- U9 pad 9: /Memory/LA11 -> AD15
Routing:
- net /Memory/LA1: track 0.00 -> 299.5 mm, vias 0 -> 2
- net /Memory/LA15: track 0.00 -> 265.7 mm, vias 0 -> 3
- net /Memory/LA13: track 0.00 -> 256.8 mm, vias 0 -> 2
- net /Memory/LA8: track 0.00 -> 252.3 mm, vias 0 -> 2
- net /Memory/LA7: track 0.00 -> 248.4 mm, vias 0 -> 2
- net /Memory/LA6: track 0.00 -> 244.4 mm, vias 0 -> 2
- net /Memory/LA4: track 0.00 -> 241.7 mm, vias 0 -> 2
- net /Memory/LA5: track 0.00 -> 239.7 mm, vias 0 -> 2
- net /Memory/LA3: track 0.00 -> 232.6 mm, vias 0 -> 2
- net /Memory/LA2: track 0.00 -> 229.7 mm, vias 0 -> 2
- net /Memory/LA14: track 0.00 -> 175.3 mm, vias 0 -> 4
- net /Memory/LA9: track 0.00 -> 171.5 mm, vias 0 -> 4
- net /Memory/LA10: track 0.00 -> 170.1 mm, vias 0 -> 4
- net /Memory/LA12: track 0.00 -> 167.7 mm, vias 0 -> 4
- net /Memory/LA11: track 0.00 -> 166.1 mm, vias 0 -> 4
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Other:
- board size 100 x 100 mm -> 366.5 x 152.2 mm
- board text added: "RAM1"
- board text added: "RAM2"
