File: 8086 board/8086 board.kicad_pcb (KiCad board)
At the start: 2 copper layers, 100 x 100 mm, 196 parts, among them J2 RM68090, J3 RGB LCD, J4 AVR-ISP-6, J5 UART, SW33 RESET, U1 P8086-2, U10 74AC373, U11 74HC138, U12 74HC138, U13 CXK58257AM, U14 IS61C256AH, U15 IS61C256AH, U16 IS61C256AH, U17 IS61C256AH, U18 IS61C3216, U19 AM29F002, U2 74AC00, U20 AM29F002, U21 28F400B5, U22 74AC373, U23 74AC373, U24 74AC373, U25 74AC373, U26 74AC373, U27 74AC373, U28 74AC373, U29 74AC373, U3 74HC14, U30 74LVC245A, U31 74LVC245A, U32 74LVC245A, U33 ATmega328P, U34 74HC595, U35 74HC595, U36 74HC595, U37 74HC165, U38 74HC165, U4 74HC02, U5 74HC02, U6 AMS1117-3.3, U7 CP2102N-Axx-xQFN28, U8 74AC373, U9 74AC373, Y1 16MHz

Commit message: initial pcb
Parts:
- removed D27, D28: LED, LED_SMD:LED_0603_1608Metric_Pad1.05x0.95mm_HandSolder
- removed DS3, DS4: 7SEG, 8086PC:2181AS
- removed RA12, RA13, RA14, RA15: 220R, Resistor_SMD:R_Array_Concave_4x0603
- removed U14, U15, U16, U17: IS61C256AH, Package_SO:TSOP-I-28_11.8x8mm_P0.55mm
- removed U18: IS61C3216, Package_SO:TSOP-II-44_10.16x18.41mm_P0.8mm
- removed U19, U20: AM29F002, Package_SO:TSOP-I-32_18.4x8mm_P0.5mm
- removed U2: 74AC00, Package_SO:SOIC-14_3.9x8.7mm_P1.27mm
- removed U21: 28F400B5, Package_SO:TSOP-I-48_18.4x12mm_P0.5mm
- removed U24, U25: 74AC373, Package_SO:SOIC-20W_7.5x12.8mm_P1.27mm
- removed U5: 74HC02, Package_SO:SOIC-14_3.9x8.7mm_P1.27mm
- added TP6: ~{B}, TestPoint:TestPoint_Pad_1.5x1.5mm, F.Cu at (423.0, 79.9)
- added U1: P8086-2, Package_DIP:DIP-40_W15.24mm, B.Cu at (-212.5, 142.0)
- added U10: 74AC573, Package_SO:TSSOP-20_4.4x6.5mm_P0.65mm, B.Cu at (-219.6, 144.5)
- added U39: 29F800BA, Package_SO:TSOP-I-48_18.4x12mm_P0.5mm, F.Cu at (-117.9, 101.6)
- added U40: IS61C6416AL, Package_SO:TSOP-II-44_10.16x18.41mm_P0.8mm, F.Cu at (-135.1, 101.4)
- added U8: 74AC573, Package_SO:TSSOP-20_4.4x6.5mm_P0.65mm, B.Cu at (-202.1, 133.4)
- added U9: 74AC573, Package_SO:TSSOP-20_4.4x6.5mm_P0.65mm, B.Cu at (-210.5, 133.4)
- DS1, DS2, JP1, JP2: moved to B.Cu
- JP3: value MEM1 -> MEM; moved to B.Cu
- TP4: value Y -> ~{A}
- U10, U22, U23, U26, U27, U28, U8, U9: value 74AC373 -> 74AC573; footprint Package_SO:SOIC-20W_7.5x12.8mm_P1.27mm -> Package_SO:TSSOP-20_4.4x6.5mm_P0.65mm
- U13: value CXK58257AM -> IS61C6416AL; footprint Package_SO:SOIC-28W_7.5x17.9mm_P1.27mm -> Package_SO:TSOP-II-44_10.16x18.41mm_P0.8mm
- U29: value 74AC373 -> 74AC573
- moved U13 586.4 mm to (-135.1, 101.4), turned to 180 degrees
- moved U1 535.2 mm to (-131.5, 141.2)
- moved U10 479.6 mm to (-138.4, 153.9)
- moved U9 477.4 mm to (-122.6, 135.1), turned to 90 degrees
- moved U8 443.4 mm to (-102.3, 135.1)
- moved RA1 272.6 mm to (127.2, 38.9)
- moved SW33 272.6 mm to (119.3, 40.6)
- moved JP3 256.7 mm to (83.3, 27.9), turned to 180 degrees
- moved JP1 254.3 mm to (84.6, 31.8), turned to 180 degrees
- moved JP2 254.3 mm to (84.6, 35.3), turned to 180 degrees
- moved U12 179.4 mm to (201.5, 124.8)
- moved U11 179.3 mm to (201.6, 116.5)
- moved R3 153.3 mm to (463.4, 16.8), turned to 90 degrees
- moved R2 150.3 mm to (460.9, 16.8), turned to 90 degrees
- moved R1 147.3 mm to (458.4, 16.8), turned to 90 degrees
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- renumbered SW8 to SW5, SW5 to SW8
Connections:
- BUS1 pad 14: ~{SEG2} -> unconnected-(BUS1-~{SEG2}-Pad14)
- BUS1 pad 16: ~{SEG3} -> unconnected-(BUS1-~{SEG3}-Pad16)
- BUS1 pad 18: ~{SEG4} -> unconnected-(BUS1-~{SEG4}-Pad18)
- BUS1 pad 20: ~{SEG5} -> unconnected-(BUS1-~{SEG5}-Pad20)
- D21 pad 2: /Memory/LED_CC -> /Memory/~{FLASH}
- D22 pad 2: /Memory/LED_CC -> /Memory/~{RAM1}
- D23 pad 2: /Memory/LED_CC -> /Memory/~{RAM2}
- D24 pad 2: /Memory/LED_CC -> GND
- J2 pad 10: ~{SEG7} -> ~{LCD}
- JP3 pad 1: /Memory/SEG1 -> GND
- JP3 pad 2: /Memory/LA19 -> +5V
- JP3 pad 3: /Memory/MEM1 -> /Memory/MEM
- RA7 pad 2: /Memory/~{LBHE} -> +5V
- RA7 pad 3: /Memory/SEG0 -> +5V
- RA7 pad 4: /Memory/SEG1 -> +5V
- SW5 pad 2: /IO/I7 -> /IO/I4
- SW8 pad 2: /IO/I4 -> /IO/I7
- U10 pad 12: /Memory/~{LBHE} -> unconnected-(U10-O7-Pad12)
- U10 pad 13: ~{BHE} -> unconnected-(U10-O6-Pad13)
- U10 pad 15: unconnected-(U10-O5-Pad15) -> /Memory/~{LBHE}
- U10 pad 16: unconnected-(U10-O6-Pad16) -> /Memory/LA19
- U10 pad 17: unconnected-(U10-D6-Pad17) -> /Memory/LA18
- U10 pad 18: unconnected-(U10-D7-Pad18) -> /Memory/LA17
- U10 pad 19: unconnected-(U10-O7-Pad19) -> /Memory/LA16
- U10 pad 2: /Memory/LA16 -> A16
- U10 pad 3: A16 -> A17
- U10 pad 4: A17 -> A18
- U10 pad 5: /Memory/LA17 -> A19
- U10 pad 6: /Memory/LA18 -> ~{BHE}
- U10 pad 7: A18 -> GND
- U10 pad 8: A19 -> GND
- U10 pad 9: /Memory/LA19 -> GND
- U11 pad 1: /Memory/LA16 -> /Memory/LA17
- U11 pad 10: ~{SEG5} -> unconnected-(U11-~{O5}-Pad10)
- U11 pad 11: ~{SEG4} -> unconnected-(U11-~{O4}-Pad11)
- U11 pad 12: ~{SEG3} -> ~{LCD}
- U11 pad 13: ~{SEG2} -> ~{MCU}
- U11 pad 14: ~{SEG1} -> /Memory/~{RAM2}
- U11 pad 15: ~{SEG0} -> /Memory/~{RAM1}
- U11 pad 2: /Memory/LA17 -> /Memory/LA18
- U11 pad 3: /Memory/LA18 -> GND
- U11 pad 7: ~{SEG7} -> unconnected-(U11-~{O7}-Pad7)
- U11 pad 9: ~{SEG6} -> unconnected-(U11-~{O6}-Pad9)
- U13 pad 1: /Memory/LA15 -> /Memory/LA16
- U13 pad 10: /Memory/LA1 -> AD3
- U13 pad 11: AD0 -> +5V
- U13 pad 12: AD1 -> GND
- U13 pad 13: AD2 -> AD4
- U13 pad 14: GND -> AD5
- U13 pad 15: AD3 -> AD6
- U13 pad 16: AD4 -> AD7
- U13 pad 17: AD5 -> ~{WR}
- U13 pad 18: AD6 -> /Memory/LA11
- U13 pad 19: AD7 -> /Memory/LA10
- U13 pad 2: /Memory/LA13 -> /Memory/LA15
- U13 pad 20: /Memory/~{SEG0L} -> /Memory/LA9
- U13 pad 21: /Memory/LA11 -> /Memory/LA8
- U13 pad 22: ~{RD} -> unconnected-(U13-NC-Pad22)
- U13 pad 23: /Memory/LA12 -> unconnected-(U13-NC-Pad23)
- U13 pad 24: /Memory/LA10 -> /Memory/LA7
- U13 pad 25: /Memory/LA9 -> /Memory/LA6
- U13 pad 26: /Memory/LA14 -> /Memory/LA5
- U13 pad 27: ~{WR} -> /Memory/LA4
- U13 pad 28: +5V -> unconnected-(U13-NC-Pad28)
- U13 pad 3: /Memory/LA8 -> /Memory/LA14
- U13 pad 4: /Memory/LA7 -> /Memory/LA13
- U13 pad 5: /Memory/LA6 -> /Memory/LA12
- U13 pad 6: /Memory/LA5 -> /Memory/~{RAM1}
- U13 pad 7: /Memory/LA4 -> AD0
- U13 pad 8: /Memory/LA3 -> AD1
- U13 pad 9: /Memory/LA2 -> AD2
- U22 pad 12: /IO/O4 -> /IO/O7
- U22 pad 13: AD4 -> /IO/O6
- U22 pad 14: AD5 -> /IO/O5
- U22 pad 15: /IO/O5 -> /IO/O4
- U22 pad 16: /IO/O6 -> /IO/O3
- U22 pad 17: AD6 -> /IO/O2
- U22 pad 18: AD7 -> /IO/O1
- U22 pad 19: /IO/O7 -> /IO/O0
- U22 pad 2: /IO/O0 -> AD0
- U22 pad 3: AD0 -> AD1
- U22 pad 4: AD1 -> AD2
- U22 pad 5: /IO/O1 -> AD3
- U22 pad 6: /IO/O2 -> AD4
- U22 pad 7: AD2 -> AD5
- U22 pad 8: AD3 -> AD6
- U22 pad 9: /IO/O3 -> AD7
- U23 pad 12: /IO/O12 -> /IO/O15
- U23 pad 13: AD12 -> /IO/O14
- U23 pad 14: AD13 -> /IO/O13
- U23 pad 15: /IO/O13 -> /IO/O12
- U23 pad 16: /IO/O14 -> /IO/O11
- U23 pad 17: AD14 -> /IO/O10
- U23 pad 18: AD15 -> /IO/O9
- U23 pad 19: /IO/O15 -> /IO/O8
- U23 pad 2: /IO/O8 -> AD8
- U23 pad 3: AD8 -> AD9
- U23 pad 4: AD9 -> AD10
- U23 pad 5: /IO/O9 -> AD11
- U23 pad 6: /IO/O10 -> AD12
- U23 pad 7: AD10 -> AD13
- U23 pad 8: AD11 -> AD14
- U23 pad 9: /IO/O11 -> AD15
- U26 pad 12: AD4 -> AD7
- U26 pad 13: /IO/I4 -> AD6
- U26 pad 14: /IO/I5 -> AD5
- U26 pad 15: AD5 -> AD4
- U26 pad 16: AD6 -> AD3
- U26 pad 17: /IO/I6 -> AD2
- U26 pad 18: /IO/I7 -> AD1
- U26 pad 19: AD7 -> AD0
- U26 pad 2: AD0 -> /IO/I0
- U26 pad 3: /IO/I0 -> /IO/I1
- U26 pad 4: /IO/I1 -> /IO/I2
- U26 pad 5: AD1 -> /IO/I3
- U26 pad 6: AD2 -> /IO/I4
- U26 pad 7: /IO/I2 -> /IO/I5
- U26 pad 8: /IO/I3 -> /IO/I6
- U26 pad 9: AD3 -> /IO/I7
- U27 pad 12: AD12 -> AD15
- U27 pad 13: /IO/I12 -> AD14
- U27 pad 14: /IO/I13 -> AD13
- U27 pad 15: AD13 -> AD12
- U27 pad 16: AD14 -> AD11
- U27 pad 17: /IO/I14 -> AD10
- U27 pad 18: /IO/I15 -> AD9
- U27 pad 19: AD15 -> AD8
- U27 pad 2: AD8 -> /IO/I8
- U27 pad 3: /IO/I8 -> /IO/I9
- U27 pad 4: /IO/I9 -> /IO/I10
- U27 pad 5: AD9 -> /IO/I11
- U27 pad 6: AD10 -> /IO/I12
- U27 pad 7: /IO/I10 -> /IO/I13
- U27 pad 8: /IO/I11 -> /IO/I14
- U27 pad 9: AD11 -> /IO/I15
- U28 pad 12: AD4 -> AD7
- U28 pad 13: /IO/I20 -> AD6
- U28 pad 14: /IO/I21 -> AD5
- U28 pad 15: AD5 -> AD4
- U28 pad 16: AD6 -> AD3
- U28 pad 17: /IO/I22 -> AD2
- U28 pad 18: /IO/I23 -> AD1
- U28 pad 19: AD7 -> AD0
- U28 pad 2: AD0 -> /IO/I16
- U28 pad 3: /IO/I16 -> /IO/I17
- U28 pad 4: /IO/I17 -> /IO/I18
- U28 pad 5: AD1 -> /IO/I19
- U28 pad 6: AD2 -> /IO/I20
- U28 pad 7: /IO/I18 -> /IO/I21
- U28 pad 8: /IO/I19 -> /IO/I22
- U28 pad 9: AD3 -> /IO/I23
- U29 pad 12: AD12 -> AD15
- U29 pad 13: /IO/I28 -> AD14
- U29 pad 14: /IO/I29 -> AD13
- U29 pad 15: AD13 -> AD12
- U29 pad 16: AD14 -> AD11
- U29 pad 17: /IO/I30 -> AD10
- U29 pad 18: /IO/I31 -> AD9
- U29 pad 19: AD15 -> AD8
- U29 pad 2: AD8 -> /IO/I24
- U29 pad 3: /IO/I24 -> /IO/I25
- U29 pad 4: /IO/I25 -> /IO/I26
- U29 pad 5: AD9 -> /IO/I27
- U29 pad 6: AD10 -> /IO/I28
- U29 pad 7: /IO/I26 -> /IO/I29
- U29 pad 8: /IO/I27 -> /IO/I30
- U29 pad 9: AD11 -> /IO/I31
- U3 pad 1: ~{SEG0} -> Net-(U3-Pad1)
- U3 pad 10: /Memory/LBHE -> Net-(TP4-Pad1)
- U3 pad 11: /Memory/~{LBHE} -> Net-(TP2-Pad1)
- U3 pad 12: ALE -> Net-(TP6-Pad1)
- U3 pad 13: Net-(U3-Pad13) -> Net-(TP3-Pad1)
- U3 pad 2: /Memory/SEG0 -> ALE
- U3 pad 4: /Memory/~{LA19} -> /Memory/~{FLASH}
- U3 pad 5: /Memory/LA0 -> Net-(U3-Pad5)
- U3 pad 6: /Memory/~{LA0} -> /IO/~{RD0}
- U3 pad 8: /Memory/SEG1 -> /IO/~{RD1}
- U3 pad 9: ~{SEG1} -> Net-(U3-Pad9)
- U32 pad 6: ~{SEG7} -> ~{LCD}
- U33 pad 32: ~{SEG6} -> ~{MCU}
- U4 pad 1: Net-(U3-Pad13) -> Net-(U3-Pad1)
- U4 pad 10: /IO/WR1 -> Net-(U3-Pad9)
- U4 pad 11: Net-(TP2-Pad1) -> ~{WR}
- U4 pad 12: Net-(TP3-Pad1) -> ~{IO0}
- U4 pad 13: Net-(TP4-Pad1) -> /IO/WR0
- U4 pad 4: /IO/WR0 -> Net-(U3-Pad5)
- U4 pad 5: ~{WR} -> ~{RD}
- U4 pad 8: ~{WR} -> ~{RD}
- U8 pad 12: /Memory/LA4 -> /Memory/LA7
- U8 pad 13: AD4 -> /Memory/LA6
- U8 pad 14: AD5 -> /Memory/LA5
- U8 pad 15: /Memory/LA5 -> /Memory/LA4
- U8 pad 16: /Memory/LA6 -> /Memory/LA3
- U8 pad 17: AD6 -> /Memory/LA2
- U8 pad 18: AD7 -> /Memory/LA1
- U8 pad 19: /Memory/LA7 -> /Memory/LA0
- U8 pad 2: /Memory/LA0 -> AD0
- U8 pad 3: AD0 -> AD1
- U8 pad 4: AD1 -> AD2
- U8 pad 5: /Memory/LA1 -> AD3
- U8 pad 6: /Memory/LA2 -> AD4
- U8 pad 7: AD2 -> AD5
- U8 pad 8: AD3 -> AD6
- U8 pad 9: /Memory/LA3 -> AD7
- U9 pad 12: /Memory/LA12 -> /Memory/LA15
- U9 pad 13: AD12 -> /Memory/LA14
- U9 pad 14: AD13 -> /Memory/LA13
- U9 pad 15: /Memory/LA13 -> /Memory/LA12
- U9 pad 16: /Memory/LA14 -> /Memory/LA11
- U9 pad 17: AD14 -> /Memory/LA10
- U9 pad 18: AD15 -> /Memory/LA9
- U9 pad 19: /Memory/LA15 -> /Memory/LA8
- U9 pad 2: /Memory/LA8 -> AD8
- U9 pad 3: AD8 -> AD9
- U9 pad 4: AD9 -> AD10
- U9 pad 5: /Memory/LA9 -> AD11
- U9 pad 6: /Memory/LA10 -> AD12
- U9 pad 7: AD10 -> AD13
- U9 pad 8: AD11 -> AD14
- U9 pad 9: /Memory/LA11 -> AD15
Routing:
- net AD0: track 0.00 -> 48.9 mm, vias 0 -> 1
- net AD1: track 0.00 -> 45.1 mm, vias 0 -> 1
- net AD2: track 0.00 -> 41.6 mm, vias 0 -> 1
- net GND: track 0.00 -> 38.5 mm
- net AD8: track 0.00 -> 36.9 mm, vias 0 -> 1
- net AD4: track 0.00 -> 36.0 mm, vias 0 -> 1
- net AD5: track 0.00 -> 35.5 mm, vias 0 -> 1
- net AD6: track 0.00 -> 35.4 mm, vias 0 -> 1
- net AD15: track 0.00 -> 35.1 mm, vias 0 -> 1
- net AD7: track 0.00 -> 35.1 mm, vias 0 -> 1
- net AD9: track 0.00 -> 32.8 mm, vias 0 -> 1
- net ~{BHE}: track 0.00 -> 30.1 mm
- net AD10: track 0.00 -> 29.8 mm, vias 0 -> 1
- net AD11: track 0.00 -> 27.3 mm, vias 0 -> 1
- net A19: track 0.00 -> 26.4 mm
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
Commit message: connect flash and ram together
Parts:
- moved U1 242.1 mm to (108.5, 109.1)
- moved U1 242.1 mm to (27.4, 109.8)
- moved U10 242.1 mm to (20.3, 112.4)
- moved U10 242.1 mm to (101.5, 121.7)
- moved U13 242.1 mm to (104.9, 69.2)
- moved U39 242.1 mm to (122.1, 69.5)
- moved U40 242.1 mm to (104.9, 69.2)
- moved U8 242.1 mm to (137.7, 103.0)
- moved U8 242.1 mm to (37.8, 101.3)
- moved U9 242.1 mm to (117.4, 103.0)
- moved U9 242.1 mm to (29.5, 101.3)
- moved JP3 47.3 mm to (130.5, 31.6)
- moved JP1 47.3 mm to (131.8, 35.5)
- moved JP2 47.3 mm to (131.8, 39.0)
- moved SW33 38.6 mm to (157.0, 32.0)
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Routing:
- net /Memory/LA16: track 11.7 -> 45.6 mm, vias 1 -> 2
- net /Memory/LA14: track 11.7 -> 45.3 mm, vias 1 -> 2
- net /Memory/LA15: track 11.7 -> 45.2 mm, vias 1 -> 2
- net /Memory/LA13: track 11.4 -> 42.5 mm, vias 1 -> 2
- net /Memory/LA12: track 12.0 -> 40.9 mm, vias 1 -> 2
- net /Memory/LA2: track 11.7 -> 40.3 mm, vias 1 -> 3
- net /Memory/LA3: track 11.6 -> 39.2 mm, vias 1 -> 3
- net AD1: track 45.1 -> 72.4 mm, vias 1 -> 2
- net /Memory/LA1: track 11.4 -> 38.4 mm, vias 1 -> 3
- net AD0: track 48.9 -> 74.5 mm, vias 1 -> 2
- net ~{RD}: track 11.9 -> 37.2 mm, vias 1 -> 3
- net AD2: track 41.6 -> 66.8 mm, vias 1 -> 2
- net AD8: track 36.9 -> 61.3 mm
- net AD3: track 26.2 -> 50.2 mm, vias 0 -> 1
- net AD4: track 36.0 -> 60.0 mm, vias 1 -> 2
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
Commit message: reduced schematic, PCB memory routed
Parts:
- removed D25, D26: LED, LED_SMD:LED_0603_1608Metric_Pad1.05x0.95mm_HandSolder
- removed DS1, DS2: 7SEG, 8086PC:2181AS
- removed JP6: D/~{C}, Jumper:SolderJumper-3_P2.0mm_Open_TrianglePad1.0x1.5mm
- removed JP7: DISP, Jumper:SolderJumper-3_P2.0mm_Open_TrianglePad1.0x1.5mm
- removed RA10, RA11, RA8, RA9: 220R, Resistor_SMD:R_Array_Concave_4x0603
- removed TP3: B, TestPoint:TestPoint_Pad_1.5x1.5mm
- removed TP4: ~{A}, TestPoint:TestPoint_Pad_1.5x1.5mm
- removed the U1 at (27.4, 109.8)
- removed the U10 at (20.3, 112.4)
- removed U22, U23: 74AC573, Package_SO:TSSOP-20_4.4x6.5mm_P0.65mm
- removed U3: 74HC14, Package_SO:SOIC-14_3.9x8.7mm_P1.27mm
- removed U4: 74HC02, Package_SO:SOIC-14_3.9x8.7mm_P1.27mm
- removed the U8 at (37.8, 101.3)
- removed the U9 at (29.5, 101.3)
- D1, D10, D11, D12, D13, D14, D15, D16, D17, D18, D19, D2, D20, D3, D4, D5, D6, D7, D8, D9, U39: moved to B.Cu
- D21: value PWR -> FLASH; moved to B.Cu
- D22: value ~{BHE} -> RAM1; moved to B.Cu
- D23: value SEG0 -> RAM2; moved to B.Cu
- D24: value SEG1 -> POWER; moved to B.Cu
- TP2: value A -> ~
- TP6: value ~{B} -> ~; moved to B.Cu
- U26: moved to F.Cu
- moved TP6 359.6 mm to (64.1, 57.5), turned to 180 degrees
- moved RA5 315.3 mm to (32.3, 68.5), turned to -90 degrees
- moved RA6 315.0 mm to (26.3, 68.5), turned to -90 degrees
- moved RA4 314.4 mm to (38.3, 68.5), turned to -90 degrees
- moved RA3 313.6 mm to (44.3, 68.5), turned to -90 degrees
- moved RA2 312.7 mm to (50.3, 68.5), turned to -90 degrees
- moved D20 308.1 mm to (24.0, 62.5), turned to 90 degrees
- moved D19 306.1 mm to (25.5, 62.5), turned to 90 degrees
- moved D18 302.9 mm to (27.0, 62.5), turned to 90 degrees
- moved D17 300.9 mm to (28.5, 62.5), turned to 90 degrees
- moved D16 298.9 mm to (30.0, 62.5), turned to 90 degrees
- moved D15 296.9 mm to (31.5, 62.5), turned to 90 degrees
- moved D14 294.9 mm to (33.0, 62.5), turned to 90 degrees
- moved D13 292.9 mm to (34.5, 62.5), turned to 90 degrees
- moved D12 289.9 mm to (36.0, 62.5), turned to 90 degrees
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Connections:
- JP3 pad 2: +5V -> /Memory/MEM
- JP3 pad 3: /Memory/MEM -> +5V
- JP4 pad 2: +3.3V -> /IO/IM0
- JP4 pad 3: /IO/IM0 -> +3.3V
- JP5 pad 1: /IO/O7 -> Net-(JP5-Pad1)
- JP5 pad 2: +3.3V -> /IO/~{LCD_RST}
- JP5 pad 3: /IO/~{LCD_RST} -> +3.3V
- RA2 pad 1: /Memory/LA0 -> Net-(D4-A)
- RA2 pad 2: /Memory/LA1 -> Net-(D3-A)
- RA2 pad 3: /Memory/LA2 -> Net-(D2-A)
- RA2 pad 4: /Memory/LA3 -> Net-(D1-A)
- RA2 pad 5: Net-(D4-A) -> /Memory/LA0
- RA2 pad 6: Net-(D3-A) -> /Memory/LA1
- RA2 pad 7: Net-(D2-A) -> /Memory/LA2
- RA2 pad 8: Net-(D1-A) -> /Memory/LA3
- RA3 pad 1: /Memory/LA4 -> Net-(D8-A)
- RA3 pad 2: /Memory/LA5 -> Net-(D7-A)
- RA3 pad 3: /Memory/LA6 -> Net-(D6-A)
- RA3 pad 4: /Memory/LA7 -> Net-(D5-A)
- RA3 pad 5: Net-(D8-A) -> /Memory/LA4
- RA3 pad 6: Net-(D7-A) -> /Memory/LA5
- RA3 pad 7: Net-(D6-A) -> /Memory/LA6
- RA3 pad 8: Net-(D5-A) -> /Memory/LA7
- RA4 pad 1: /Memory/LA8 -> Net-(D12-A)
- RA4 pad 2: /Memory/LA9 -> Net-(D11-A)
- RA4 pad 3: /Memory/LA10 -> Net-(D10-A)
- RA4 pad 4: /Memory/LA11 -> Net-(D9-A)
- RA4 pad 5: Net-(D12-A) -> /Memory/LA8
- RA4 pad 6: Net-(D11-A) -> /Memory/LA9
- RA4 pad 7: Net-(D10-A) -> /Memory/LA10
- RA4 pad 8: Net-(D9-A) -> /Memory/LA11
- RA5 pad 1: /Memory/LA12 -> Net-(D16-A)
- RA5 pad 2: /Memory/LA13 -> Net-(D15-A)
- RA5 pad 3: /Memory/LA14 -> Net-(D14-A)
- RA5 pad 4: /Memory/LA15 -> Net-(D13-A)
- RA5 pad 5: Net-(D16-A) -> /Memory/LA12
- RA5 pad 6: Net-(D15-A) -> /Memory/LA13
- RA5 pad 7: Net-(D14-A) -> /Memory/LA14
- RA5 pad 8: Net-(D13-A) -> /Memory/LA15
- RA6 pad 1: /Memory/LA16 -> Net-(D20-A)
- RA6 pad 2: /Memory/LA17 -> Net-(D19-A)
- RA6 pad 3: /Memory/LA18 -> Net-(D18-A)
- RA6 pad 4: /Memory/LA19 -> Net-(D17-A)
- RA6 pad 5: Net-(D20-A) -> /IO/D/~{C}
- RA6 pad 6: Net-(D19-A) -> /Memory/LA17
- RA6 pad 7: Net-(D18-A) -> /Memory/LA18
- RA6 pad 8: Net-(D17-A) -> /Memory/LA19
- RA7 pad 1: +5V -> Net-(D24-A)
- RA7 pad 2: +5V -> Net-(D23-A)
- RA7 pad 3: +5V -> Net-(D22-A)
- RA7 pad 4: +5V -> Net-(D21-A)
- RA7 pad 5: Net-(D24-A) -> +5V
- RA7 pad 6: Net-(D23-A) -> +5V
- RA7 pad 7: Net-(D22-A) -> +5V
- RA7 pad 8: Net-(D21-A) -> +5V
- TP2 pad 1: Net-(TP2-Pad1) -> Net-(JP5-Pad1)
- TP6 pad 1: Net-(TP6-Pad1) -> Net-(U39-RY/~{BY})
- U10 pad 12: unconnected-(U10-O7-Pad12) -> /Memory/~{LBHE}
- U10 pad 13: unconnected-(U10-O6-Pad13) -> /Memory/LA19
- U10 pad 14: unconnected-(U10-O5-Pad14) -> /Memory/LA18
- U10 pad 15: /Memory/~{LBHE} -> /Memory/LA17
- U10 pad 16: /Memory/LA19 -> /IO/D/~{C}
- U10 pad 17: /Memory/LA18 -> unconnected-(U10-O2-Pad17)
- U10 pad 18: /Memory/LA17 -> unconnected-(U10-O1-Pad18)
- U10 pad 19: /Memory/LA16 -> unconnected-(U10-O0-Pad19)
- U10 pad 2: A16 -> GND
- U10 pad 3: A17 -> GND
- U10 pad 4: A18 -> GND
- U10 pad 5: A19 -> A16
- U10 pad 6: ~{BHE} -> A17
- U10 pad 7: GND -> A18
- U10 pad 8: GND -> A19
- U10 pad 9: GND -> ~{BHE}
- U13 pad 1: /Memory/LA16 -> /IO/D/~{C}
- U39 pad 1: /Memory/LA16 -> /IO/D/~{C}
- U40 pad 1: /Memory/LA16 -> /IO/D/~{C}
Routing:
- net /IO/D/~{C}: track 0.00 -> 91.5 mm, vias 0 -> 5
- net ~{WR}: track 11.2 -> 95.2 mm, vias 1 -> 4
- net /Memory/LA0: track 11.4 -> 67.8 mm, vias 1 -> 3
- net /Memory/LA18: track 0.00 -> 54.3 mm, vias 0 -> 2
- net /Memory/LA15: track 45.2 -> 91.2 mm, vias 2 -> 5
- net /Memory/LA16: track 45.6 -> 0.00 mm, vias 2 -> 0
- net +5V: track 14.8 -> 58.8 mm, vias 2 -> 5
- net /Memory/LA13: track 42.5 -> 86.0 mm, vias 2 -> 5
- net /Memory/LA12: track 40.9 -> 84.2 mm, vias 2 -> 5
- net /Memory/LA14: track 45.3 -> 87.6 mm, vias 2 -> 5
- net /Memory/LA17: track 0.00 -> 41.6 mm, vias 0 -> 2
- net /Memory/LA3: track 39.2 -> 79.0 mm, vias 3 -> 4
- net AD15: track 50.1 -> 89.8 mm, vias 1 -> 5
- net /Memory/LA11: track 25.0 -> 64.6 mm, vias 2 -> 3
- net AD11: track 47.4 -> 85.0 mm, vias 1 -> 3
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- added copper zone on F.Cu, net +5V
- added copper zone on B.Cu, net GND
Other:
- board size 100 x 100 mm -> 267.7 x 110.7 mm

Commit message: PCB: initial layout
Parts:
- removed BUS1: 8086 BUS, Connector_PinHeader_2.54mm:PinHeader_2x24_P2.54mm_Vertical
- removed J2: RM68090, 8086PC:RM68090 RGB LCD module
- removed TP2: ~, TestPoint:TestPoint_Pad_1.5x1.5mm
- added BUS2: ~, Connector_PinHeader_2.54mm:PinHeader_2x16_P2.54mm_Vertical, B.Cu at (261.0, 18.2)
- added U2: 74HC32, Package_SO:TSSOP-14_4.4x5mm_P0.65mm, F.Cu at (251.0, 50.4)
- C1, C2, C3, C4, C5, C6, C7, R1, R10, R2, R3, R4, R5, R9, RA16, RA17, RA18, RA19, RA20, RA21, RA22, RA23, TP1, U26, U27, U28, U29, U33, Y1: moved to B.Cu
- SW33: moved to F.Cu
- U11, U12, U37, U38: footprint Package_SO:SOIC-16_3.9x9.9mm_P1.27mm -> Package_SO:TSSOP-16_4.4x5mm_P0.65mm
- U34, U35, U36: footprint Package_SO:SOIC-16_3.9x9.9mm_P1.27mm -> Package_SO:TSSOP-16_4.4x5mm_P0.65mm; moved to B.Cu
- moved JP2 229.1 mm to (251.9, 58.4), turned to 90 degrees
- moved U1 227.6 mm to (247.0, 33.5), turned to 90 degrees
- moved D20 225.0 mm to (249.0, 58.3), turned to -90 degrees
- moved U10 223.6 mm to (246.9, 42.8), turned to -90 degrees
- moved D19 222.0 mm to (247.5, 58.3), turned to -90 degrees
- moved RA6 221.0 mm to (246.7, 52.3), turned to 90 degrees
- moved D18 219.0 mm to (246.0, 58.3), turned to -90 degrees
- moved D17 216.0 mm to (244.5, 58.3), turned to -90 degrees
- moved D16 213.0 mm to (243.0, 58.3), turned to -90 degrees
- moved D15 210.0 mm to (241.5, 58.3), turned to -90 degrees
- moved RA5 209.1 mm to (240.7, 52.3), turned to 90 degrees
- moved D14 207.0 mm to (240.0, 58.3), turned to -90 degrees
- moved D13 204.0 mm to (238.5, 58.3), turned to -90 degrees
- moved D12 201.0 mm to (237.0, 58.3), turned to -90 degrees
- moved U9 200.0 mm to (234.9, 42.8), turned to -90 degrees
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Connections:
- JP5 pad 1: Net-(JP5-Pad1) -> unconnected-(JP5-Pad1)
- U12 pad 10: ~{IO5} -> unconnected-(U12-~{O5}-Pad10)
- U12 pad 11: ~{IO4} -> unconnected-(U12-~{O4}-Pad11)
- U12 pad 12: ~{IO3} -> unconnected-(U12-~{O3}-Pad12)
- U12 pad 13: ~{IO2} -> unconnected-(U12-~{O2}-Pad13)
- U12 pad 7: ~{IO7} -> unconnected-(U12-~{O7}-Pad7)
- U12 pad 9: ~{IO6} -> unconnected-(U12-~{O6}-Pad9)
Routing:
- net /Memory/~{LBHE}: track 11.4 -> 132.5 mm
- net READY: track 0.00 -> 68.2 mm, vias 0 -> 1
- net /CPUALE: track 0.00 -> 65.8 mm, vias 0 -> 1
- net AD0: track 48.7 -> 105.5 mm, vias 2 -> 3
- net AD2: track 52.5 -> 105.1 mm, vias 2 -> 3
- net AD1: track 50.7 -> 102.1 mm, vias 2 -> 3
- net AD4: track 55.4 -> 104.3 mm, vias 2 -> 3
- net AD3: track 53.0 -> 100.3 mm, vias 2 -> 3
- net M\~{IO}: track 0.00 -> 46.9 mm
- net AD6: track 57.2 -> 101.7 mm, vias 3 -> 4
- net AD5: track 56.7 -> 100.5 mm, vias 3 -> 4
- net HLDA: track 0.00 -> 41.8 mm
- net AD7: track 61.1 -> 98.3 mm, vias 2 -> 3
- net AD8: track 68.2 -> 104.5 mm, vias 3 -> 4
- net HOLD: track 0.00 -> 36.2 mm
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Other:
- board size 267.7 x 110.7 mm -> 100 x 100 mm
- board text added: "A0"
- board text added: "A19"
