File: 8086 board/8086 board.kicad_pcb (KiCad board)
At the start: 2 copper layers, 100 x 100 mm, 162 parts, among them J3 RGB LCD, J4 AVR-ISP-6, J5 UART, SW33 RESET, U1 P8086-2, U10 74AC573, U11 74HC138, U12 74HC138, U13 IS61C6416AL, U2 74HC32, U26 74AC573, U27 74AC573, U28 74AC573, U29 74AC573, U30 74LVC245A, U31 74LVC245A, U32 74LVC245A, U33 ATmega328P, U34 74HC595, U35 74HC595, U36 74HC595, U37 74HC165, U38 74HC165, U39 29F800BA, U40 IS61C6416AL, U6 AMS1117-3.3, U7 CP2102N-Axx-xQFN28, U8 74AC573, U9 74AC573, Y1 16MHz

Commit message: PCB: more layout work. some schematic changes.
Parts:
- removed C32, C33, C34, C35, C36, C37, C38, C39, C40, C41, C42, C43: 1uF, Capacitor_SMD:C_0603_1608Metric_Pad1.08x0.95mm_HandSolder
- removed the JP1 at (194.2, 60.5)
- removed the JP3 at (200.4, 60.3)
- removed the R4 at (252.6, 109.9)
- removed the R5 at (260.2, 109.9)
- removed the U7 at (256.8, 104.3)
- added H1: ~, MountingHole:MountingHole_3.2mm_M3, F.Cu at (189.8, 18.5)
- added H2: ~, MountingHole:MountingHole_3.2mm_M3, F.Cu at (259.8, 18.5)
- added H3: ~, MountingHole:MountingHole_3.2mm_M3, F.Cu at (189.8, 68.5)
- added H4: ~, MountingHole:MountingHole_3.2mm_M3, F.Cu at (259.8, 68.5)
- added J2: USB, Connector_USB:USB_C_Receptacle_GCT_USB4105-xx-A_16P_TopMnt_Horizontal, B.Cu at (272.4, 67.8)
- added SW34: MEM_BANK, Button_Switch_SMD:SW_SPDT_PCM12, F.Cu at (185.3, 88.0)
- added U4: CH340C, Package_SO:SOIC-16_3.9x9.9mm_P1.27mm, B.Cu at (263.8, 79.2)
- J1: renamed from BUS2; value ~ -> Conn_02x16_Odd_Even
- J3, U2: moved to B.Cu
- JP1: renamed from JP4; footprint Jumper:SolderJumper-3_P2.0mm_Open_TrianglePad1.0x1.5mm -> Jumper:SolderJumper-3_P1.3mm_Bridged12_RoundedPad1.0x1.5mm; moved to B.Cu
- JP2: renamed from JP5; footprint Jumper:SolderJumper-3_P2.0mm_Open_TrianglePad1.0x1.5mm -> Jumper:SolderJumper-3_P1.3mm_Bridged12_RoundedPad1.0x1.5mm; moved to B.Cu
- JP3: renamed from JP2; footprint Jumper:SolderJumper-2_P1.3mm_Open_TrianglePad1.0x1.5mm -> Jumper:SolderJumper-2_P1.3mm_Bridged_RoundedPad1.0x1.5mm
- R4: renamed from R6; moved to B.Cu
- R5: renamed from R7; moved to B.Cu
- R6: renamed from R8; moved to B.Cu
- SW1, SW10, SW11, SW12, SW13, SW14, SW15, SW16, SW17, SW18, SW19, SW2, SW20, SW21, SW22, SW23, SW24, SW25, SW26, SW27, SW28, SW29, SW3, SW30, SW31, SW32, SW33, SW4, SW5, SW6, SW7, SW8, SW9: footprint 8086PC:SW_Push_1P1T_NO_6x6mm_H9.5mm -> 8086PC:SW_Push_6x6x5mm
- U17: renamed from U30; moved to B.Cu
- U18: renamed from U31; moved to B.Cu
- U19: renamed from U32; moved to B.Cu
- U21: renamed from U34; moved to F.Cu
- U22: renamed from U35; moved to F.Cu
- U23: renamed from U36; moved to F.Cu
- U24: renamed from U37; moved to B.Cu
- U25: renamed from U38; moved to B.Cu
- moved JP2 116.8 mm to (262.3, 58.2), turned to 180 degrees
- moved U17 110.4 mm to (260.8, 45.8)
- moved U18 110.4 mm to (260.8, 38.5)
- moved U19 110.4 mm to (260.8, 53.1)
- moved J3 109.7 mm to (252.1, 43.7)
- moved R4 107.7 mm to (258.6, 34.1)
- moved R6 107.7 mm to (258.6, 30.8)
- moved R5 107.7 mm to (258.6, 32.4)
- moved JP1 102.6 mm to (252.3, 29.2), turned to 0 degrees
- moved D23 65.3 mm to (190.5, 63.2)
- moved D22 60.6 mm to (194.9, 63.3)
- moved J5 55.8 mm to (253.2, 101.1), turned to 0 degrees
- moved C10 49.6 mm to (153.9, 27.8)
- moved C13 49.6 mm to (153.9, 35.3)
- moved C16 49.6 mm to (153.9, 42.8)
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- renumbered J5 to J4, J4 to J5, R10 to R7, RA18 to RA10, RA19 to RA11, RA20 to RA12, RA21 to RA13, RA22 to RA14, RA23 to RA15, RA16 to RA8, RA17 to RA9, TP6 to TP2, U39 to U10, U40 to U11, U13 to U12, U26 to U13, U27 to U14, U28 to U15, U29 to U16, U33 to U20, U6 to U3, U8 to U5, U9 to U6, U10 to U7, U11 to U8, U12 to U9
Connections:
- C4 pad 1: Net-(U7-VDD) -> GND
- C4 pad 2: GND -> Net-(U4-V3)
- J1 pad 10: AD3 -> A17
- J1 pad 11: AD4 -> AD14
- J1 pad 12: AD5 -> AD15
- J1 pad 13: AD6 -> AD12
- J1 pad 14: AD7 -> AD13
- J1 pad 15: AD8 -> AD10
- J1 pad 16: AD9 -> AD11
- J1 pad 17: AD10 -> AD8
- J1 pad 18: AD11 -> AD9
- J1 pad 19: AD12 -> AD6
- J1 pad 20: AD13 -> AD7
- J1 pad 21: AD14 -> AD4
- J1 pad 22: AD15 -> AD5
- J1 pad 23: A16 -> AD2
- J1 pad 24: A17 -> AD3
- J1 pad 25: A18 -> AD0
- J1 pad 26: A19 -> AD1
- J1 pad 7: AD0 -> A18
- J1 pad 8: AD1 -> A19
- J1 pad 9: AD2 -> A16
- J3 pad 38: Net-(J3-IM0) -> /IO/IM0
- J5 pad 3: /Microcontroller/SPI_SCK -> GND
- JP1 pad 1: GND -> +3.3V
- JP1 pad 3: +3.3V -> GND
- JP2 pad 1: unconnected-(JP5-Pad1) -> +3.3V
- JP2 pad 3: +3.3V -> unconnected-(JP2-Pad3)
- U10 pad 11: /Memory/~{WRP} -> ~{WR}
- U10 pad 16: /Memory/MEM -> Net-(SW34-B)
- U13 pad 12: AD7 -> AD0
- U13 pad 13: AD6 -> AD1
- U13 pad 14: AD5 -> AD2
- U13 pad 15: AD4 -> AD3
- U13 pad 16: AD3 -> AD4
- U13 pad 17: AD2 -> AD5
- U13 pad 18: AD1 -> AD6
- U13 pad 19: AD0 -> AD7
- U13 pad 2: /IO/I0 -> /IO/I7
- U13 pad 3: /IO/I1 -> /IO/I6
- U13 pad 4: /IO/I2 -> /IO/I5
- U13 pad 5: /IO/I3 -> /IO/I4
- U13 pad 6: /IO/I4 -> /IO/I3
- U13 pad 7: /IO/I5 -> /IO/I2
- U13 pad 8: /IO/I6 -> /IO/I1
- U13 pad 9: /IO/I7 -> /IO/I0
- U15 pad 12: AD7 -> AD0
- U15 pad 13: AD6 -> AD1
- U15 pad 14: AD5 -> AD2
- U15 pad 15: AD4 -> AD3
- U15 pad 16: AD3 -> AD4
- U15 pad 17: AD2 -> AD5
- U15 pad 18: AD1 -> AD6
- U15 pad 19: AD0 -> AD7
- U15 pad 2: /IO/I16 -> /IO/I23
- U15 pad 3: /IO/I17 -> /IO/I22
- U15 pad 4: /IO/I18 -> /IO/I21
- U15 pad 5: /IO/I19 -> /IO/I20
- U15 pad 6: /IO/I20 -> /IO/I19
- U15 pad 7: /IO/I21 -> /IO/I18
- U15 pad 8: /IO/I22 -> /IO/I17
- U15 pad 9: /IO/I23 -> /IO/I16
- U17 pad 11: /IO/DB7 -> /IO/DB0
- U17 pad 12: /IO/DB6 -> /IO/DB1
- U17 pad 13: /IO/DB5 -> /IO/DB2
- U17 pad 14: /IO/DB4 -> /IO/DB3
- U17 pad 15: /IO/DB3 -> /IO/DB4
- U17 pad 16: /IO/DB2 -> /IO/DB5
- U17 pad 17: /IO/DB1 -> /IO/DB6
- U17 pad 18: /IO/DB0 -> /IO/DB7
- U17 pad 2: AD0 -> AD7
- U17 pad 3: AD1 -> AD6
- U17 pad 4: AD2 -> AD5
- U17 pad 5: AD3 -> AD4
- U17 pad 6: AD4 -> AD3
- U17 pad 7: AD5 -> AD2
- U17 pad 8: AD6 -> AD1
- U17 pad 9: AD7 -> AD0
- U18 pad 11: /IO/DB15 -> /IO/DB8
- U18 pad 12: /IO/DB14 -> /IO/DB9
- U18 pad 13: /IO/DB13 -> /IO/DB10
- U18 pad 14: /IO/DB12 -> /IO/DB11
- U18 pad 15: /IO/DB11 -> /IO/DB12
- U18 pad 16: /IO/DB10 -> /IO/DB13
- U18 pad 17: /IO/DB9 -> /IO/DB14
- U18 pad 18: /IO/DB8 -> /IO/DB15
- U18 pad 2: AD8 -> AD15
- U18 pad 3: AD9 -> AD14
- U18 pad 4: AD10 -> AD13
- U18 pad 5: AD11 -> AD12
- U18 pad 6: AD12 -> AD11
- U18 pad 7: AD13 -> AD10
- U18 pad 8: AD14 -> AD9
- U18 pad 9: AD15 -> AD8
- U19 pad 11: Net-(J3-~{RD}) -> unconnected-(U19-B7-Pad11)
- U19 pad 12: Net-(J3-~{WR}) -> unconnected-(U19-B6-Pad12)
- U19 pad 13: Net-(J3-D/~{C}) -> unconnected-(U19-B5-Pad13)
- U19 pad 15: unconnected-(U32-B3-Pad15) -> Net-(J3-D/~{C})
- U19 pad 16: unconnected-(U32-B2-Pad16) -> Net-(J3-~{WR})
- U19 pad 17: Net-(J3-IM0) -> Net-(J3-~{RD})
- U19 pad 3: /IO/IM0 -> ~{RD}
- U19 pad 4: unconnected-(U32-A2-Pad4) -> ~{WR}
- U19 pad 5: unconnected-(U32-A3-Pad5) -> /IO/D/~{C}
- U19 pad 7: /IO/D/~{C} -> unconnected-(U19-A5-Pad7)
- U19 pad 8: ~{WR} -> unconnected-(U19-A6-Pad8)
- U19 pad 9: ~{RD} -> unconnected-(U19-A7-Pad9)
- U20 pad 12: /Microcontroller/RCLK_SH/~{LD} -> GND
- U20 pad 17: /Microcontroller/SPI_SCK -> GND
- U21 pad 11: /Microcontroller/SPI_SCK -> GND
- U21 pad 12: /Microcontroller/RCLK_SH/~{LD} -> GND
- U22 pad 11: /Microcontroller/SPI_SCK -> GND
- U22 pad 12: /Microcontroller/RCLK_SH/~{LD} -> GND
- U23 pad 11: /Microcontroller/SPI_SCK -> GND
- U23 pad 12: /Microcontroller/RCLK_SH/~{LD} -> GND
- U23 pad 7: unconnected-(U36-QH-Pad7) -> ~{BHE}
- U24 pad 1: /Microcontroller/RCLK_SH/~{LD} -> unconnected-(U24-SH/~{LD}-Pad1)
- U24 pad 2: /Microcontroller/SPI_SCK -> unconnected-(U24-CLK-Pad2)
- U25 pad 1: /Microcontroller/RCLK_SH/~{LD} -> GND
- U25 pad 2: /Microcontroller/SPI_SCK -> GND
Routing:
- net +5V: track 68.5 -> 438.1 mm
- net AD14: track 100.1 -> 248.5 mm, vias 3 -> 5
- net AD15: track 111.2 -> 251.9 mm, vias 3 -> 7
- net AD13: track 97.6 -> 235.4 mm, vias 3 -> 5
- net AD12: track 99.0 -> 233.7 mm, vias 3 -> 5
- net AD6: track 101.7 -> 223.7 mm, vias 4 -> 5
- net AD7: track 98.3 -> 219.6 mm, vias 3 -> 4
- net AD0: track 105.5 -> 225.7 mm, vias 3 -> 5
- net AD4: track 104.3 -> 221.7 mm, vias 3 -> 4
- net AD5: track 100.5 -> 216.3 mm, vias 4 -> 5
- net AD2: track 105.1 -> 218.4 mm, vias 3 -> 4
- net AD11: track 103.6 -> 214.7 mm, vias 3 -> 6
- net AD3: track 100.3 -> 211.3 mm, vias 3 -> 4
- net AD1: track 102.1 -> 211.7 mm, vias 3 -> 4
- net AD10: track 102.9 -> 210.2 mm, vias 3 -> 5
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Other:
- board size 100 x 100 mm -> 94 x 90 mm
- board text added: "1"
- board text added: "2.4{dblquote}"
- board text added: "2.8{dblquote}"
- board text added: "3.5{dblquote}"
- board text added: "40"
- board text added: "Reset"

Commit message: PCB: different layout
Parts:
- added R8: 10k, Resistor_SMD:R_0603_1608Metric_Pad0.98x0.95mm_HandSolder, B.Cu at (118.3, 44.0)
- added TP3: XL, TestPoint:TestPoint_Pad_1.5x1.5mm, B.Cu at (187.8, 83.0)
- added TP4: YU, TestPoint:TestPoint_Pad_1.5x1.5mm, B.Cu at (187.8, 85.5)
- added TP5: XR, TestPoint:TestPoint_Pad_1.5x1.5mm, B.Cu at (190.3, 83.0)
- added TP6: YD, TestPoint:TestPoint_Pad_1.5x1.5mm, B.Cu at (190.3, 85.5)
- C25, C26, C27, C28, C29, C30, C31, SW34, U21, U22, U23: moved to B.Cu
- J1: value Conn_02x16_Odd_Even -> 8086 bus
- R9: value 1k -> 10k
- U24, U25: moved to F.Cu
- moved D20 208.4 mm to (46.9, 112.5)
- moved D19 205.5 mm to (48.4, 112.5)
- moved RA6 204.3 mm to (49.2, 107.5)
- moved D18 202.6 mm to (49.9, 112.5)
- moved D17 199.7 mm to (51.4, 112.5)
- moved D16 196.8 mm to (52.9, 112.5)
- moved D15 193.9 mm to (54.4, 112.5)
- moved RA5 192.8 mm to (55.2, 107.5)
- moved D14 191.0 mm to (55.9, 112.5)
- moved D13 188.2 mm to (57.4, 112.5)
- moved D12 185.3 mm to (58.9, 112.5)
- moved D11 182.4 mm to (60.4, 112.5)
- moved RA4 181.2 mm to (61.2, 107.5)
- moved JP3 180.4 mm to (79.0, 112.7)
- moved D10 179.5 mm to (61.9, 112.5)
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Connections:
- J1 pad 1: ~{RD} -> A18
- J1 pad 10: A17 -> AD11
- J1 pad 11: AD14 -> AD8
- J1 pad 12: AD15 -> AD9
- J1 pad 13: AD12 -> AD6
- J1 pad 14: AD13 -> AD7
- J1 pad 15: AD10 -> AD4
- J1 pad 16: AD11 -> AD5
- J1 pad 17: AD8 -> AD2
- J1 pad 18: AD9 -> AD3
- J1 pad 19: AD6 -> AD0
- J1 pad 2: HOLD -> A19
- J1 pad 20: AD7 -> AD1
- J1 pad 21: AD4 -> BUSALE
- J1 pad 22: AD5 -> ~{BHE}
- J1 pad 23: AD2 -> M\~{IO}
- J1 pad 24: AD3 -> READY
- J1 pad 25: AD0 -> HLDA
- J1 pad 26: AD1 -> ~{WR}
- J1 pad 27: BUSALE -> ~{RD}
- J1 pad 28: ~{BHE} -> HOLD
- J1 pad 3: HLDA -> A16
- J1 pad 4: ~{WR} -> A17
- J1 pad 5: M\~{IO} -> AD14
- J1 pad 6: READY -> AD15
- J1 pad 7: A18 -> AD12
- J1 pad 8: A19 -> AD13
- J1 pad 9: A16 -> AD10
- J3 pad 1: unconnected-(J3-TOUCH_XL-Pad1) -> /IO/XL
- J3 pad 2: unconnected-(J3-TOUCH_YU-Pad2) -> /IO/YU
- J3 pad 3: unconnected-(J3-TOUCH_XR-Pad3) -> /IO/XR
- J3 pad 4: unconnected-(J3-TOUCH_YD-Pad4) -> /IO/YD
- J5 pad 3: GND -> /Microcontroller/SPI_SCK
- U17 pad 11: /IO/DB0 -> /IO/DB7
- U17 pad 12: /IO/DB1 -> /IO/DB6
- U17 pad 13: /IO/DB2 -> /IO/DB5
- U17 pad 14: /IO/DB3 -> /IO/DB4
- U17 pad 15: /IO/DB4 -> /IO/DB3
- U17 pad 16: /IO/DB5 -> /IO/DB2
- U17 pad 17: /IO/DB6 -> /IO/DB1
- U17 pad 18: /IO/DB7 -> /IO/DB0
- U17 pad 2: AD7 -> AD0
- U17 pad 3: AD6 -> AD1
- U17 pad 4: AD5 -> AD2
- U17 pad 5: AD4 -> AD3
- U17 pad 6: AD3 -> AD4
- U17 pad 7: AD2 -> AD5
- U17 pad 8: AD1 -> AD6
- U17 pad 9: AD0 -> AD7
- U18 pad 11: /IO/DB8 -> /IO/DB15
- U18 pad 12: /IO/DB9 -> /IO/DB14
- U18 pad 13: /IO/DB10 -> /IO/DB13
- U18 pad 14: /IO/DB11 -> /IO/DB12
- U18 pad 15: /IO/DB12 -> /IO/DB11
- U18 pad 16: /IO/DB13 -> /IO/DB10
- U18 pad 17: /IO/DB14 -> /IO/DB9
- U18 pad 18: /IO/DB15 -> /IO/DB8
- U18 pad 2: AD15 -> AD8
- U18 pad 3: AD14 -> AD9
- U18 pad 4: AD13 -> AD10
- U18 pad 5: AD12 -> AD11
- U18 pad 6: AD11 -> AD12
- U18 pad 7: AD10 -> AD13
- U18 pad 8: AD9 -> AD14
- U18 pad 9: AD8 -> AD15
- U19 pad 11: unconnected-(U19-B7-Pad11) -> Net-(J3-~{RESET})
- U19 pad 12: unconnected-(U19-B6-Pad12) -> Net-(J3-~{RD})
- U19 pad 13: unconnected-(U19-B5-Pad13) -> Net-(J3-~{WR})
- U19 pad 14: Net-(J3-~{CS}) -> Net-(J3-D/~{C})
- U19 pad 15: Net-(J3-D/~{C}) -> Net-(J3-~{CS})
- U19 pad 16: Net-(J3-~{WR}) -> unconnected-(U19-B2-Pad16)
- U19 pad 17: Net-(J3-~{RD}) -> unconnected-(U19-B1-Pad17)
- U19 pad 18: Net-(J3-~{RESET}) -> unconnected-(U19-B0-Pad18)
- U19 pad 2: /IO/~{LCD_RST} -> unconnected-(U19-A0-Pad2)
- U19 pad 3: ~{RD} -> unconnected-(U19-A1-Pad3)
- U19 pad 4: ~{WR} -> unconnected-(U19-A2-Pad4)
- U19 pad 5: /IO/D/~{C} -> ~{LCD}
- U19 pad 6: ~{LCD} -> /IO/D/~{C}
- U19 pad 7: unconnected-(U19-A5-Pad7) -> ~{WR}
- U19 pad 8: unconnected-(U19-A6-Pad8) -> ~{RD}
- U19 pad 9: unconnected-(U19-A7-Pad9) -> /IO/~{LCD_RST}
- U20 pad 12: GND -> /Microcontroller/RCLK_SH/~{LD}
- U20 pad 17: GND -> /Microcontroller/SPI_SCK
- U21 pad 11: GND -> /Microcontroller/SPI_SCK
- U21 pad 12: GND -> /Microcontroller/RCLK_SH/~{LD}
- U22 pad 11: GND -> /Microcontroller/SPI_SCK
- U22 pad 12: GND -> /Microcontroller/RCLK_SH/~{LD}
- U23 pad 11: GND -> /Microcontroller/SPI_SCK
- U23 pad 12: GND -> /Microcontroller/RCLK_SH/~{LD}
- U24 pad 1: unconnected-(U24-SH/~{LD}-Pad1) -> /Microcontroller/RCLK_SH/~{LD}
- U24 pad 2: unconnected-(U24-CLK-Pad2) -> /Microcontroller/SPI_SCK
- U25 pad 1: GND -> /Microcontroller/RCLK_SH/~{LD}
- U25 pad 2: GND -> /Microcontroller/SPI_SCK
- U5 pad 12: /Memory/LA7 -> /Memory/LA15
- U5 pad 13: /Memory/LA6 -> /Memory/LA14
- U5 pad 14: /Memory/LA5 -> /Memory/LA13
- U5 pad 15: /Memory/LA4 -> /Memory/LA12
- U5 pad 6: AD4 -> AD12
- U5 pad 7: AD5 -> AD13
- U5 pad 8: AD6 -> AD14
- U5 pad 9: AD7 -> AD15
- U6 pad 12: /Memory/LA15 -> /Memory/LA11
- U6 pad 13: /Memory/LA14 -> /Memory/LA10
- U6 pad 14: /Memory/LA13 -> /Memory/LA9
- U6 pad 15: /Memory/LA12 -> /Memory/LA8
- U6 pad 16: /Memory/LA11 -> /Memory/LA7
- U6 pad 17: /Memory/LA10 -> /Memory/LA6
- U6 pad 18: /Memory/LA9 -> /Memory/LA5
- U6 pad 19: /Memory/LA8 -> /Memory/LA4
- U6 pad 2: AD8 -> AD4
- U6 pad 3: AD9 -> AD5
- U6 pad 4: AD10 -> AD6
- U6 pad 5: AD11 -> AD7
- U6 pad 6: AD12 -> AD8
- U6 pad 7: AD13 -> AD9
- U6 pad 8: AD14 -> AD10
- U6 pad 9: AD15 -> AD11
Routing:
- net +5V: track 438.1 -> 60.1 mm
- net ~{WR}: track 141.2 -> 22.9 mm, vias 7 -> 2
- net AD14: track 248.5 -> 135.2 mm, vias 5 -> 3
- net A16: track 142.9 -> 35.1 mm, vias 2 -> 0
- net ~{BHE}: track 104.5 -> 0.00 mm, vias 2 -> 0
- net AD13: track 235.4 -> 140.2 mm, vias 5 -> 3
- net AD15: track 251.9 -> 156.8 mm, vias 7 -> 2
- net A17: track 130.0 -> 36.7 mm, vias 2 -> 0
- net A18: track 121.0 -> 30.7 mm, vias 2 -> 0
- net AD12: track 233.7 -> 150.4 mm, vias 5 -> 3
- net A19: track 113.3 -> 30.0 mm, vias 2 -> 0
- net AD6: track 223.7 -> 144.7 mm, vias 5 -> 3
- net AD7: track 219.6 -> 141.0 mm, vias 4 -> 3
- net READY: track 77.6 -> 0.00 mm, vias 2 -> 0
- net /Memory/~{LBHE}: track 100.8 -> 25.9 mm, vias 3 -> 1
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- removed copper zone on F.Cu, net +5V
- removed copper zone on B.Cu, net GND
Other:
- outline, holes or cut-outs redrawn
- board text added: "hold reset button while programming!"
- board text added: "locked"
- board text removed: "1"
- board text removed: "2.4{dblquote}"
- board text removed: "2.8{dblquote}"
- board text removed: "3.5{dblquote}"
- board text removed: "Alt"
- board text removed: "Backspace"
- board text removed: "Ctrl"
- board text removed: "Enter"
- board text removed: "Reset"
- board text removed: "Shift"
- board text removed: "Space"
