File: 8086 board/memory.kicad_sch (KiCad schematic)
At the start: 10 parts, among them U17 AM29F002, U18 AM29F002, U19 CXK58257AM, U20 IS61C3216, U21 IS61C256AH, U22 IS61C256AH, U30 IS61C256AH, U31 IS61C256AH, U9 28F400

Commit message: refactoring schematic files and structure
Parts:
- added JP2: ~, symbol 8086PC:jumper_3
- added U23: 74HC14, Package_SO:SOIC-14_3.9x8.7mm_P1.27mm, symbol 8086PC:74HC14
- added U3, U4, U5: 74HC373, Package_SO:SOIC-20W_7.5x12.8mm_P1.27mm, symbol 8086PC:74AC373
- added U6, U7: 74LS138, Package_SO:SOIC-16_3.9x9.9mm_P1.27mm, symbol 8086PC:74HC138
- added U8: 74AC00, Package_SO:SOIC-14_3.9x8.7mm_P1.27mm, symbol 8086PC:74AC00
Connections:
- net +5V: now also U3.20 (VCC), U4.20 (VCC), U5.20 (VCC), U6.16 (VCC), U6.6 (E3), U7.16 (VCC)
- net AD0: now also U5.3 (D0)
- net AD1: now also U5.4 (D1)
- net AD10: now also U3.7 (D2)
- net AD11: now also U3.8 (D3)
- net AD12: now also U3.13 (D4)
- net AD13: now also U3.14 (D5)
- net AD14: now also U3.17 (D6)
- net AD15: now also U3.18 (D7)
- net AD2: now also U5.7 (D2)
- net AD3: now also U5.8 (D3)
- net AD4: now also U5.13 (D4)
- net AD5: now also U5.14 (D5)
- net AD6: now also U5.17 (D6)
- net AD7: now also U5.18 (D7)
- net AD8: now also U3.3 (D0)
- net AD9: now also U3.4 (D1)
- net GND: now also U3.1 (~{OE}), U3.10 (GND), U4.1 (~{OE}), U4.10 (GND), U5.1 (~{OE}), U5.10 (GND), U6.8 (GND), U7.8 (GND)
- net LA0: now also U23.1, U5.2 (O0)
- net LA1: now also U5.5 (O1), U6.1 (A0)
- net LA10: now also U3.6 (O2)
- net LA11: now also U3.9 (O3)
- net LA12: now also U3.12 (O4)
- net LA13: now also U3.15 (O5)
- net LA14: now also U3.16 (O6)
- net LA15: now also U3.19 (O7)
- net LA16: now also U4.2 (O0), U7.1 (A0)
- net LA17: now also U4.5 (O1), U7.2 (A1)
- net LA18: now also U4.6 (O2), U7.3 (A2)
- net LA19: now also JP2.3 (B), U23.3, U4.9 (O3), U7.4 (~{E1}), U7.5 (~{E2})
- net LA2: now also U5.6 (O2), U6.2 (A1)
- net LA3: now also U5.9 (O3), U6.3 (A2)
- net LA4: now also U5.12 (O4)
- net LA5: now also U5.15 (O5)
- net LA6: now also U5.16 (O6)
- net LA7: now also U5.19 (O7)
- net LA8: now also U3.2 (O0)
- net LA9: now also U3.5 (O1)
- net ~{LA19}: now also U23.4
- net ~{LBHE}: now also U23.11
- net ~{MEM1H}: now also U8.11
- net ~{MEM1L}: now also U8.8
- net ~{SEG0H}: now also U8.6
- net ~{SEG0L}: now also U8.3
- net ~{SEG0}: now also U23.9, U7.15 (~{O0})
- net ~{SEG1}: now also U23.5, U7.14 (~{O1})
- new net: JP2.2 (C), U8.10, U8.12
- new net A16: U4.3 (D0)
- new net A17: U4.4 (D1)
- new net A18: U4.7 (D2)
- new net A19: U4.8 (D3)
- new net ALE: U3.11 (LE), U4.11 (LE), U5.11 (LE)
- new net LBHE: U23.10, U4.12 (O4), U8.13, U8.5
- new net M/~{IO}: U6.4 (~{E1}), U6.5 (~{E2}), U7.6 (E3)
- new net SEG0: U23.8, U8.2, U8.4
- new net SEG1: JP2.1 (A), U23.6
- new net ~{BHE}: U4.13 (D4)
- new net ~{IO0}: U6.15 (~{O0})
- new net ~{IO1}: U6.14 (~{O1})
- new net ~{IO2}: U6.13 (~{O2})
- new net ~{IO3}: U6.12 (~{O3})
- new net ~{IO4}: U6.11 (~{O4})
- new net ~{IO5}: U6.10 (~{O5})
- new net ~{IO6}: U6.9 (~{O6})
- new net ~{IO7}: U6.7 (~{O7})
- new net ~{LA0}: U23.2, U8.1, U8.9
- new net ~{SEG2}: U7.13 (~{O2})
- new net ~{SEG3}: U7.12 (~{O3})
- new net ~{SEG4}: U7.11 (~{O4})
- new net ~{SEG5}: U7.10 (~{O5})
- new net ~{SEG6}: U7.9 (~{O6})
- new net ~{SEG7}: U7.7 (~{O7})
- no-connect marks 0 -> 6
Other:
- note added: "AD[0-7]"
- note added: "AD[16-19], BHE"
- note added: "AD[8-15]"
- note added: "Address latching"
- note added: "Are the 2 hex inverters pin and footprint compatible??"
- note added: "CS LOGIC"
- note added: "IO[0-7]"
- note added: "SEG[0-7]"
- note added: "SEG[0-7] IO[0-7] 3-8 decoders"
- moved on the sheet: JP1

Commit message: better schematic. initial pcb layout
Parts:
- removed JP1: Write Protect, symbol Jumper:Jumper_2_Bridged
- removed JP2: ~, symbol 8086PC:jumper_3
- added D33: A4, LED_SMD:LED_0603_1608Metric_Pad1.05x0.95mm_HandSolder, symbol 8086PC:LED_small
- added D34: A5, LED_SMD:LED_0603_1608Metric_Pad1.05x0.95mm_HandSolder, symbol 8086PC:LED_small
- added D35: A6, LED_SMD:LED_0603_1608Metric_Pad1.05x0.95mm_HandSolder, symbol 8086PC:LED_small
- added D36: A7, LED_SMD:LED_0603_1608Metric_Pad1.05x0.95mm_HandSolder, symbol 8086PC:LED_small
- added D37: A8, LED_SMD:LED_0603_1608Metric_Pad1.05x0.95mm_HandSolder, symbol 8086PC:LED_small
- added D38: A9, LED_SMD:LED_0603_1608Metric_Pad1.05x0.95mm_HandSolder, symbol 8086PC:LED_small
- added D39: A10, LED_SMD:LED_0603_1608Metric_Pad1.05x0.95mm_HandSolder, symbol 8086PC:LED_small
- added D40: A11, LED_SMD:LED_0603_1608Metric_Pad1.05x0.95mm_HandSolder, symbol 8086PC:LED_small
- added D41: A12, LED_SMD:LED_0603_1608Metric_Pad1.05x0.95mm_HandSolder, symbol 8086PC:LED_small
- added D42: A13, LED_SMD:LED_0603_1608Metric_Pad1.05x0.95mm_HandSolder, symbol 8086PC:LED_small
- added D43: A14, LED_SMD:LED_0603_1608Metric_Pad1.05x0.95mm_HandSolder, symbol 8086PC:LED_small
- added D44: A15, LED_SMD:LED_0603_1608Metric_Pad1.05x0.95mm_HandSolder, symbol 8086PC:LED_small
- added D45: A16, LED_SMD:LED_0603_1608Metric_Pad1.05x0.95mm_HandSolder, symbol 8086PC:LED_small
- added D46: A17, LED_SMD:LED_0603_1608Metric_Pad1.05x0.95mm_HandSolder, symbol 8086PC:LED_small
- added D47: A18, LED_SMD:LED_0603_1608Metric_Pad1.05x0.95mm_HandSolder, symbol 8086PC:LED_small
- added D48: A0, LED_SMD:LED_0603_1608Metric_Pad1.05x0.95mm_HandSolder, symbol 8086PC:LED_small
- added D49: A1, LED_SMD:LED_0603_1608Metric_Pad1.05x0.95mm_HandSolder, symbol 8086PC:LED_small
- added D50: A2, LED_SMD:LED_0603_1608Metric_Pad1.05x0.95mm_HandSolder, symbol 8086PC:LED_small
- added D51: A3, LED_SMD:LED_0603_1608Metric_Pad1.05x0.95mm_HandSolder, symbol 8086PC:LED_small
- added D52: A19, LED_SMD:LED_0603_1608Metric_Pad1.05x0.95mm_HandSolder, symbol 8086PC:LED_small
- added D53: ~{BHE}, LED_SMD:LED_0603_1608Metric_Pad1.05x0.95mm_HandSolder, symbol 8086PC:LED_small
- added D54: SEG0, LED_SMD:LED_0603_1608Metric_Pad1.05x0.95mm_HandSolder, symbol 8086PC:LED_small
- added D55: SEG1, LED_SMD:LED_0603_1608Metric_Pad1.05x0.95mm_HandSolder, symbol 8086PC:LED_small
- added D56: PWR, LED_SMD:LED_0603_1608Metric_Pad1.05x0.95mm_HandSolder, symbol 8086PC:LED_small
- added JP1: Write Protect, symbol 8086PC:Jumper_2_Bridged
- added JP2: LEDs, symbol 8086PC:Jumper_2_Bridged
- added JP5: MEM1, symbol 8086PC:SolderJumper
- added RA1, RA2, RA3, RA4, RA5, RA6: 220R, Resistor_SMD:R_Array_Concave_4x0603, symbol 8086PC:R_Array_4
- U24: renamed from U9; value 28F400 -> 28F400B5
- U3: renamed from U5; value 74HC373 -> 74AC373
- U4: renamed from U3; value 74HC373 -> 74AC373
- U5: renamed from U4; value 74HC373 -> 74AC373
- U6: renamed from U7; value 74LS138 -> 74HC138
- U7: renamed from U6; value 74LS138 -> 74HC138
- renumbered U19 to U17, U22 to U18, U30 to U19, U31 to U21, U18 to U22, U17 to U26, U21 to U9
Connections:
- net +5V: now also RA6.1
- net GND: now also JP2.3 (B)
- net LA0: now also RA1.1
- net LA1: now also RA1.2
- net LA10: now also RA3.3
- net LA11: now also RA3.4
- net LA12: now also RA4.1
- net LA13: now also RA4.2
- net LA14: now also RA4.3
- net LA15: now also RA4.4
- net LA16: now also RA5.1
- net LA17: now also RA5.2
- net LA18: now also RA5.3
- net LA19: now also JP5.2, RA5.4
- net LA2: now also RA1.3
- net LA3: now also RA1.4
- net LA4: now also RA2.1
- net LA5: now also RA2.2
- net LA6: now also RA2.3
- net LA7: now also RA2.4
- net LA8: now also RA3.1
- net LA9: now also RA3.2
- net LBHE: no longer U5.12 (O4)
- net SEG0: now also RA6.3
- net SEG1: now also JP5.1, RA6.4
- net ~{LBHE}: now also U5.12 (O4), RA6.2
- net ~{WRP}: now also JP1.3 (B)
- net ~{WR}: now also JP1.1 (A)
- net MEM1: now reaches U8.10, U8.12
- net MEM1: now also JP5.3
- net M/~{IO} renamed M\~{IO}
- new net: D51.1 (A), RA1.5
- new net: D50.1 (A), RA1.6
- new net: D49.1 (A), RA1.7
- new net: D48.1 (A), RA1.8
- new net: D47.1 (A), RA5.6
- new net: D54.1 (A), RA6.6
- new net: D36.1 (A), RA2.5
- new net: D56.1 (A), RA6.8
- new net: D53.1 (A), RA6.7
- new net: D52.1 (A), RA5.5
- new net: D40.1 (A), RA3.5
- new net: D35.1 (A), RA2.6
- new net: D34.1 (A), RA2.7
- new net: D33.1 (A), RA2.8
- new net: D46.1 (A), RA5.7
- new net: D45.1 (A), RA5.8
- new net: D43.1 (A), RA4.6
- new net: D39.1 (A), RA3.6
- new net: D38.1 (A), RA3.7
- new net: D44.1 (A), RA4.5
- new net: D42.1 (A), RA4.7
- new net: D41.1 (A), RA4.8
- new net: D37.1 (A), RA3.8
- new net: D55.1 (A), RA6.5
- new net LED_EN: D33.2 (K), D34.2 (K), D35.2 (K), D36.2 (K), D37.2 (K), D38.2 (K), D39.2 (K), D40.2 (K), D41.2 (K), D42.2 (K), D43.2 (K), D44.2 (K), D45.2 (K), D46.2 (K), D47.2 (K), D48.2 (K), D49.2 (K), D50.2 (K), D51.2 (K), D52.2 (K), D53.2 (K), D54.2 (K), D55.2 (K), D56.2 (K), JP2.1 (A)
Other:
- note added: "Alternative IC - different footprint"
- note added: "Flash - 64kB"
- note added: "Global 8086 bus"
- note added: "Jumpers"
- note added: "LEDs"
- note removed: "64k Flash"
- note removed: "Alternative IC (different footprint)"
- note removed: "Are the 2 hex inverters pin and footprint compatible??"
- note removed: "Flash"
- note removed: "Flash access LED, SRAM access LED"
- moved on the sheet: U17, U18, U19, U21, U22, U23A, U23B, U23C, U23D, U23E, U26, U3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

Commit message: Schematic finished! (some footprint assignments are still needed)
Parts:
- JP1, JP2: footprint (none) -> Jumper:SolderJumper-2_P1.3mm_Open_TrianglePad1.0x1.5mm
- JP3: renamed from JP5; footprint (none) -> Jumper:SolderJumper-3_P2.0mm_Open_TrianglePad1.0x1.5mm
- renumbered D48 to D1, D38 to D10, D39 to D11, D40 to D12, D41 to D13, D42 to D14, D43 to D15, D44 to D16, D45 to D17, D46 to D18, D47 to D19, D49 to D2, D52 to D20, D56 to D21, D53 to D22, D54 to D23, D55 to D24, D50 to D3, D51 to D4, D33 to D5, D34 to D6, D35 to D7, D36 to D8, D37 to D9, RA1 to RA2, RA2 to RA3, RA3 to RA4, RA4 to RA5, RA5 to RA6, RA6 to RA7, U5 to U10, U6 to U11, U7 to U12, U17 to U13, U9 to U14, U18 to U15, U19 to U16, U21 to U17, U20 to U18, U22 to U19, U8 to U2, U26 to U20, U24 to U21, U23 to U3, U3 to U8, U4 to U9
Connections:
- net GND: now also JP2.2 (B); no longer JP2.3 (B)
- net LA0: now also U3.5; no longer U3.1
- net SEG0: now also U3.2; no longer U3.8
- net SEG1: now also U3.8; no longer U3.6
- net ~{LA0}: now also U3.6; no longer U3.2
- net ~{SEG0}: now also U3.1; no longer U3.9
- net ~{SEG1}: now also U3.9; no longer U3.5
- net ~{WRP}: now also JP1.2 (B); no longer JP1.3 (B)
- net LED_EN renamed LED_CC
Other:
- note added: "RAM1 - 64kB"
- note added: "RAM2 - 64kB"
- note removed: "RAM1"
- note removed: "RAM2"
- moved on the sheet: D1, D10, D11, D12, D13, D14, D15, D16, D17, D18, D19, D2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
