File: 8086 board/io.kicad_sch (KiCad schematic)
At the start: 63 parts, among them J2 RGB LCD, U2 74HC32, U3 74LVC245A, U4 74LVC245A, U5 74LVC245A, U6 74AC573, U7 74AC573, U8 74AC573, U9 74AC573

Commit message: PCB: move to kicad 8
Parts:
- gave numbers to parts that had none: 5
- renumbered H3 to H2, H2 to H3, TP1 to TP2, TP1 to TP3, TP1 to TP4, U2 to U22
