File: 8086 board/microcontroller.kicad_sch (KiCad schematic)
At the start: 25 parts, among them J2 USB, U15 74HC595, U16 74HC595, U17 74HC595, U18 ATmega328P, U23 74HC165, U24 74HC165, U26 CH340C, Y1 16MHz

Commit message: PCB: move to kicad 8
Parts:
- gave numbers to parts that had none: 2
- renumbered C5 to C18, C44 to C28, J2 to J5, R1 to R10, R3 to R8, R2 to R9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
